File: applications_din/out_8x_16A_bistab_4MU/out_8x_16A_bistab_4MU_v2.1.0_kicad/out_8x_16A_bistab.kicad_sch (KiCad schematic)
At the start: 30 parts, among them IC1 ULN2803A, IC2 ULN2803A, J1 Screw_Terminal_01x02, K1 HFE20-1-024-1HD504, K2 HFE20-1-024-1HD504, K3 HFE20-1-024-1HD504, K4 HFE20-1-024-1HD504, K5 HFE20-1-024-1HD504, K6 HFE20-1-024-1HD504, K7 HFE20-1-024-1HD504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

Commit message: rename and move out 8x 16A bistab 2.1 kicad
Parts:
- C1, C2: footprint app_out_8x_16A_bistab_4MU_BOT_v2.0.0:E3,5-8 -> out_8x_16A_bistab:E3,5-8
- C3, C4: footprint app_out_8x_16A_bistab_4MU_BOT_v2.0.0:C1206 -> out_8x_16A_bistab:C1206
- IC1, IC2: footprint app_out_8x_16A_bistab_4MU_BOT_v2.0.0:SO18W -> out_8x_16A_bistab:SO18W
- JP2: footprint app_out_8x_16A_bistab_4MU_BOT_v2.0.0:2X13SMD -> out_8x_16A_bistab:2X13SMD; symbol app_out_8x_16A_bistab_4MU_BOT_v2.0.0-eagle-import:PINHD-2X13_2.54-SMD -> out_8x_16A_bistab-eagle-import:PINHD-2X13_2.54-SMD
- K1, K2, K3, K4, K5, K6, K7, K8: footprint app_out_8x_16A_bistab_4MU_BOT_v2.0.0:HFE20-3-504 -> out_8x_16A_bistab:HFE20-3-504; symbol app_out_8x_16A_bistab_4MU_BOT_v2.0.0-eagle-import:HFE20-1-024-1HD504 -> out_8x_16A_bistab-eagle-import:HFE20-1-024-1HD504
- R1, R2, R3, R4: footprint app_out_8x_16A_bistab_4MU_BOT_v2.0.0:M1206 -> out_8x_16A_bistab:M1206
- X1, X2, X3, X4, X5, X6, X7, X8: footprint app_out_8x_16A_bistab_4MU_BOT_v2.0.0:W237-132 -> out_8x_16A_bistab:W237-132; symbol app_out_8x_16A_bistab_4MU_BOT_v2.0.0-eagle-import:W237-02P -> out_8x_16A_bistab-eagle-import:W237-02P
