File: applications_din/in-out_2x-2x_2MU/top_led_btn_2MU_TOP/top_led_btn_2MU_TOP/top_led_btn_2MU_TOP.kicad_pcb (KiCad board)
At the start: 2 copper layers, 32 x 42 mm, 17 parts, among them J2 Conn_01x08_Pin, SW1 SW_PROG, SW2 SW_OUTA, SW3 SW_OUTB

Commit message: update
Parts:
- moved J2 20.1 mm to (126.7, 102.6), turned to 180 degrees
- moved R1 5.08 mm to (113.0, 88.9)
- moved R2 5.08 mm to (119.4, 99.1)
- moved R4 2.84 mm to (121.9, 90.2)
- moved R6 2.84 mm to (121.9, 92.7)
- moved R5 1.27 mm to (121.9, 95.2)
- moved D4 1.02 mm to (105.2, 78.7)
- moved D5 1.02 mm to (111.5, 78.7)
- moved D7 1.02 mm to (124.2, 78.7)
- moved D6 1.02 mm to (117.9, 78.7)
- turned D1 to -90 degrees
Connections:
- R4 pad 2: Net-(J2-Pin_3) -> Net-(J2-Pin_6)
- R5 pad 1: Net-(J2-Pin_6) -> Net-(J2-Pin_3)
Routing:
- net Net-(D2-K): track 22.8 -> 8.80 mm, vias 1 -> 0
- net Net-(D3-K): track 39.7 -> 26.6 mm, vias 1 -> 0
- net Net-(D1-K): track 34.2 -> 22.1 mm
- net Net-(D6-K): track 19.0 -> 25.1 mm
- net +3V3: track 30.3 -> 35.9 mm, vias 0 -> 1
- net Net-(D4-K): track 29.0 -> 26.4 mm
- net Net-(D4-A): track 32.3 -> 34.3 mm
- net Net-(D1-A): track 2.55 -> 3.31 mm
- net Net-(J2-Pin_4): track 4.17 -> 4.75 mm
- net Net-(J2-Pin_3): track 4.17 -> 4.75 mm
- net GND: vias 0 -> 10
Other:
- board text added: "OUT A"
- board text added: "OUT B"
- board text added: "PROG"
- board text added: "top_led_btn_2MU_TOP v1.0"
- board text removed: "top_led_tbn_2MU_TOP v1.0"

Commit message: update in-out_4x-2x_2MU - final for now
Parts:
- SW1, SW2, SW3: footprint Button_Switch_SMD:SW_SPST_CK_RS282G05A3 -> Button_Switch_SMD:SW_SPST_Omron_B3FS-100xP
- moved D1 2.27 mm to (114.6, 86.9), turned to 0 degrees
- moved R1 1.61 mm to (114.6, 89.4), turned to 180 degrees
- moved SW1 0.76 mm to (109.0, 88.9)
- moved SW2 0.76 mm to (121.2, 108.0), turned to -90 degrees
- moved SW3 0.76 mm to (109.0, 108.0), turned to -90 degrees
- moved R4 0.25 mm to (121.9, 89.9)
- moved R5 0.25 mm to (121.9, 95.5)
- moved J2 0.12 mm to (126.5, 102.6)
Routing:
- net Net-(D1-K): track 22.1 -> 17.4 mm
- net Net-(D6-K): track 25.1 -> 27.6 mm
- net Net-(D3-K): track 26.6 -> 28.8 mm
- net +3V3: track 35.9 -> 34.4 mm
- net Net-(D2-K): track 8.80 -> 9.83 mm
Other:
- board text added: "switch alternativ PTS636 SKG25J SMTR LFS https://eu.mouser.com/ProductDetail/CK/PTS636-SKG25J-SMTR-LFS"

Commit message: final for manufacturing
Parts:
- R4, R5, R6: value 470 -> 1k
Changed lines of the file:
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@@
 			)
 		)
-		(property "Value" "470"
+		(property "Value" "1k"
 			(at 0 1.65 0)
 			(layer "F.Fab")
@@
 			)
 		)
-		(property "Value" "470"
+		(property "Value" "1k"
 			(at 0 1.65 180)
 			(layer "F.Fab")
@@
 			)
 		)
-		(property "Value" "470"
+		(property "Value" "1k"
 			(at 0 1.65 0)
 			(layer "F.Fab")
