File: applications_din/in-out_2x-2x_2MU/top_led_btn_2MU_TOP/top_led_btn_2MU_TOP/top_led_btn_2MU_TOP.kicad_sch (KiCad schematic)
At the start: 17 parts, among them J2 Conn_01x08_Pin, SW1 SW_PROG, SW2 SW_OUTA, SW3 SW_OUTB

Commit message: update
Connections:
- net at J2.3 (Pin_3): now also R5.1; no longer R4.2
- net at J2.6 (Pin_6): now also R4.2; no longer R5.1
Changed lines of the file:
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@@
+	(wire
+		(pts
+			(xy 53.34 62.23) (xy 53.34 91.44)
+		)
+		(stroke
+			(width 0)
+			(type default)
+		)
+	)
 	(wire
 		(pts
@@
 	(wire
 		(pts
-			(xy 39.37 62.23) (xy 57.15 62.23)
+			(xy 39.37 62.23) (xy 53.34 62.23)
 		)
 		(stroke
@@
 	(wire
 		(pts
-			(xy 53.34 54.61) (xy 53.34 91.44)
-		)
-		(stroke
-			(width 0)
-			(type default)
-		)
-	)
-	(wire
-		(pts
 			(xy 60.96 54.61) (xy 64.77 54.61)
 		)
@@
 	(wire
 		(pts
-			(xy 57.15 62.23) (xy 57.15 81.28)
+			(xy 57.15 54.61) (xy 57.15 81.28)
 		)
 		(stroke
@@
 	(wire
 		(pts
-			(xy 39.37 54.61) (xy 53.34 54.61)
+			(xy 39.37 54.61) (xy 57.15 54.61)
 		)
 		(stroke
@@
 		(fields_autoplaced yes)
 		(property "Reference" "SW1"
-			(at 68.453 58.4778 90)
+			(at 68.58 58.4199 90)
 			(effects
 				(font
@@
 		)
 		(property "Value" "SW_PROG"
-			(at 68.453 60.9021 90)
+			(at 68.58 60.9599 90)
 			(effects
 				(font
@@
 		(fields_autoplaced yes)
 		(property "Reference" "R1"
-			(at 66.548 34.3478 0)
+			(at 67.31 34.2899 0)
 			(effects
 				(font
@@
 		)
 		(property "Value" "1k"
-			(at 66.548 36.7721 0)
+			(at 67.31 36.8299 0)
 			(effects
 				(font
@@
 		(fields_autoplaced yes)
 		(property "Reference" "J2"
-			(at 34.925 45.3093 0)
+			(at 34.925 44.45 0)
 			(effects
 				(font
@@
 		)
 		(property "Value" "Conn_01x08_Pin"
-			(at 34.925 47.7336 0)
+			(at 34.925 46.99 0)
 			(effects
 				(font
@@
 		)
 		(property "Value" "GND"
-			(at 93.98 67.945 90)
+			(at 91.44 66.0399 0)
 			(effects
 				(font
@@
 		)
 		(property "Value" "+3V3"
-			(at 64.77 27.6169 0)
-			(effects
-				(font
-					(size 1.27 1.27)
-				)
+			(at 67.31 30.4799 0)
+			(effects
+				(font
+					(size 1.27 1.27)
+				)
+				(justify left)
 			)
 		)
@@
 		)
 		(property "Value" "+3V3"
-			(at 80.01 28.575 90)
+			(at 82.55 30.4799 0)
 			(effects
 				(font
@@
 		(fields_autoplaced yes)
 		(property "Reference" "D5"
-			(at 67.6275 83.8665 0)
+			(at 67.6275 82.55 0)
 			(effects
 				(font
@@
 		)
 		(property "Value" "LED_IN2"
-			(at 67.6275 86.2908 0)
+			(at 67.6275 85.09 0)
 			(effects
 				(font
@@
 		(fields_autoplaced yes)
 		(property "Reference" "R6"
-			(at 47.7521 83.8778 0)
+			(at 46.99 83.8199 0)
 			(effects
 				(font
@@
 		)
 		(property "Value" "470"
-			(at 47.7521 86.3021 0)
+			(at 46.99 86.3599 0)
 			(effects
 				(font
@@
 		(fields_autoplaced yes)
 		(property "Reference" "D3"
-			(at 96.901 43.5553 90)
+			(at 97.79 43.4974 90)
 			(effects
 				(font
@@
 		)
 		(property "Value" "LED_OUTB"
-			(at 96.901 45.9796 90)
+			(at 97.79 46.0374 90)
 			(effects
 				(font
@@
 		(fields_autoplaced yes)
 		(property "Reference" "R2"
-			(at 81.788 34.3478 0)
+			(at 82.55 34.2899 0)
 			(effects
 				(font
@@
 		)
 		(property "Value" "1k"
-			(at 81.788 36.7721 0)
+			(at 82.55 36.8299 0)
 			(effects
 				(font
@@
 		(fields_autoplaced yes)
 		(property "Reference" "D4"
-			(at 64.4525 97.8591 0)
+			(at 64.4525 100.33 0)
 			(effects
 				(font
@@
 		)
 		(property "Value" "LED_IN1"
-			(at 64.4525 100.2834 0)
+			(at 64.4525 102.87 0)
 			(effects
 				(font
@@
 		)
 		(property "Value" "GND"
-			(at 42.545 59.69 90)
+			(at 43.18 59.6899 90)
 			(effects
 				(font
@@
 		(fields_autoplaced yes)
 		(property "Reference" "D7"
-			(at 75.8825 97.8591 0)
+			(at 75.8825 99.06 0)
 			(effects
 				(font
@@
 		)
 		(property "Value" "LED_IN4"
-			(at 75.8825 100.2834 0)
+			(at 75.8825 101.6 0)
 			(effects
 				(font
@@
 		(fields_autoplaced yes)
 		(property "Reference" "D1"
-			(at 67.691 43.5553 90)
+			(at 68.58 43.4974 90)
 			(effects
 				(font
@@
 		)
 		(property "Value" "LED_PROG"
-			(at 67.691 45.9796 90)
+			(at 68.58 46.0374 90)
 			(effects
 				(font
@@
 		(fields_autoplaced yes)
 		(property "Reference" "R3"
-			(at 95.758 34.3478 0)
+			(at 96.52 34.2899 0)
 			(effects
 				(font
@@
 		)
 		(property "Value" "1k"
-			(at 95.758 36.7721 0)
+			(at 96.52 36.8299 0)
 			(effects
 				(font
@@
 		)
 		(property "Value" "GND"
-			(at 64.77 68.9031 0)
+			(at 64.77 69.85 0)
 			(effects
 				(font
@@
 		)
 		(property "Value" "+3V3"
-			(at 42.545 64.77 90)
+			(at 43.18 64.7699 90)
 			(effects
 				(font
@@
 		)
 		(property "Value" "GND"
-			(at 80.01 67.945 90)
+			(at 77.47 66.0399 0)
 			(effects
 				(font
@@
 		(fields_autoplaced yes)
 		(property "Reference" "SW3"
-			(at 97.663 58.4778 90)
+			(at 97.79 58.4199 90)
 			(effects
 				(font
@@
 		)
 		(property "Value" "SW_OUTB"
-			(at 97.663 60.9021 90)
+			(at 97.79 60.9599 90)
 			(effects
 				(font
@@
 		(fields_autoplaced yes)
 		(property "Reference" "R5"
-			(at 58.928 83.8778 0)
+			(at 59.69 83.8199 0)
 			(effects
 				(font
@@
 		)
 		(property "Value" "470"
-			(at 58.928 86.3021 0)
+			(at 59.69 86.3599 0)
 			(effects
 				(font
@@
 		(fields_autoplaced yes)
 		(property "Reference" "D2"
-			(at 82.931 43.5553 90)
+			(at 83.82 43.4974 90)
 			(effects
 				(font
@@
 		)
 		(property "Value" "LED_OUTA"
-			(at 82.931 45.9796 90)
+			(at 83.82 46.0374 90)
 			(effects
 				(font
@@
 		(fields_autoplaced yes)
 		(property "Reference" "SW2"
-			(at 83.693 58.4778 90)
+			(at 83.82 58.4199 90)
 			(effects
 				(font
@@
 		)
 		(property "Value" "SW_OUTA"
-			(at 83.693 60.9021 90)
+			(at 83.82 60.9599 90)
 			(effects
 				(font
@@
 		(fields_autoplaced yes)
 		(property "Reference" "D6"
-			(at 79.0575 83.8665 0)
+			(at 79.0575 82.55 0)
 			(effects
 				(font
@@
 		)
 		(property "Value" "LED_IN3"
-			(at 79.0575 86.2908 0)
+			(at 79.0575 85.09 0)
 			(effects
 				(font
@@
 		)
 		(property "Value" "+3V3"
-			(at 93.98 28.575 90)
+			(at 96.52 30.4799 0)
 			(effects
 				(font
@@
 		(fields_autoplaced yes)
 		(property "Reference" "R4"
-			(at 55.118 94.0378 0)
+			(at 55.88 93.9799 0)
 			(effects
 				(font
@@
 		)
 		(property "Value" "470"
-			(at 55.118 96.4621 0)
-			(effects
-				(font
+			(at 55.88 96.5199 0)
+			(effects
+				(font

Commit message: update in-out_4x-2x_2MU - final for now
Parts:
- SW1, SW2, SW3: footprint Button_Switch_SMD:SW_SPST_CK_RS282G05A3 -> Button_Switch_SMD:SW_SPST_Omron_B3FS-100xP
Changed lines of the file:
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@@
 			)
 		)
-		(property "Footprint" "Button_Switch_SMD:SW_SPST_CK_RS282G05A3"
+		(property "Footprint" "Button_Switch_SMD:SW_SPST_Omron_B3FS-100xP"
 			(at 69.85 59.69 0)
 			(effects
@@
 			)
 		)
-		(property "Footprint" "Button_Switch_SMD:SW_SPST_CK_RS282G05A3"
+		(property "Footprint" "Button_Switch_SMD:SW_SPST_Omron_B3FS-100xP"
 			(at 99.06 59.69 0)
 			(effects
@@
 			)
 		)
-		(property "Footprint" "Button_Switch_SMD:SW_SPST_CK_RS282G05A3"
+		(property "Footprint" "Button_Switch_SMD:SW_SPST_Omron_B3FS-100xP"
 			(at 85.09 59.69 0)
 			(effects

Commit message: final for manufacturing
Parts:
- R4, R5, R6: value 470 -> 1k
Changed lines of the file:
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@@
 			)
 		)
-		(property "Value" "470"
+		(property "Value" "1k"
 			(at 46.99 86.3599 0)
 			(effects
@@
 			)
 		)
-		(property "Value" "470"
+		(property "Value" "1k"
 			(at 59.69 86.3599 0)
 			(effects
@@
 			)
 		)
-		(property "Value" "470"
+		(property "Value" "1k"
 			(at 55.88 96.5199 0)
 			(effects
