File: applications_din/out_8x_16A_bistab_4MU/out_8x_16A_bistab_4MU_v2.3.0_kicad/out_8x_16A_bistab.kicad_pcb (KiCad board)
At the start: 2 copper layers, 86.5 x 68 mm, 27 parts, among them IC1 ULN2803A, IC2 ULN2803A, J1 Screw_Terminal_01x02, J2 Conn_01x04_Socket, J3 Conn_01x04_Socket, J4 Conn_01x04_Socket, J5 Conn_01x04_Socket, K1 HFE20-1-024-1HD504, K2 HFE20-1-024-1HD504, K3 HFE20-1-024-1HD504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

Commit message: update out_8x_16A_bistab_4MU_v2.3.0_kicad - final for now
Parts:
- moved R4 7.07 mm to (146.3, 122.6), turned to 90 degrees
- moved R3 3.97 mm to (148.3, 122.6), turned to 90 degrees
- moved R2 2.52 mm to (150.4, 122.6), turned to 90 degrees
- moved D1 1.48 mm to (178.3, 131.3)
- moved C1 1.09 mm to (118.9, 131.1)
- moved C2 1.02 mm to (172.0, 132.2)
- moved JP2 1.02 mm to (146.8, 131.3)
- moved JP1 0.40 mm to (124.2, 136.7)
Routing:
- net GND: track 113.7 -> 0.00 mm, vias 1 -> 15
- net /+3V3: track 15.8 -> 12.4 mm
- net /IO16: track 7.11 -> 9.40 mm
- net /APP_SEL: track 16.6 -> 18.8 mm
- net /IO3: track 9.26 -> 11.5 mm
- net /IO12: track 6.63 -> 8.77 mm
- net /IO8: track 5.11 -> 6.73 mm
- net /IO1: track 5.11 -> 6.73 mm
- net /IO10: track 9.29 -> 10.8 mm
- net /IO4: track 5.93 -> 7.26 mm
- net /IO6: track 6.05 -> 7.17 mm
- net /O5: track 51.9 -> 52.8 mm
- net /EIB_DC: track 39.6 -> 40.4 mm
- net VBUS: track 25.2 -> 25.8 mm
- added copper zone on B.Cu, net GND
- added copper zone on F.Cu, net GND
Other:
- board text added: "www.selfbus.org Schaltaktor out8 16A V2.3 kicad"
- board text removed: "www.selfbus.org Schaltaktor out8 16A V2.3"

Commit message: update all stuff
Parts:
- J1: value Screw_Terminal_01x02 -> EIB_WAGO_243-211
- J6: renamed from JP2; footprint Connector_PinHeader_2.54mm:PinHeader_2x13_P2.54mm_Vertical_SMD -> Connector_IDC:IDC-Header_2x13_P2.54mm_Vertical_SMD
Routing:
- net VBUS: track 25.8 -> 26.3 mm

Commit message: finally standardize selected parts on all boards
Parts:
- added D2: 12V, Diode_SMD:D_MiniMELF, F.Cu at (122.7, 136.1)
- J2, J3, J4, J5: value Conn_01x04_Socket -> Con_230V
- R1: footprint Resistor_SMD:R_0805_2012Metric -> Resistor_SMD:R_1206_3216Metric
- moved JP1 4.82 mm to (122.7, 132.1)
- moved C1 2.79 mm to (116.1, 131.1)
- moved R1 0.53 mm to (126.0, 131.6)
Routing:
- net VDD: track 174.5 -> 179.1 mm
- net /EIB_DC: track 40.7 -> 41.7 mm

Commit message: final for manufacturing
Parts:
- J1: value EIB_WAGO_243-211 -> WAGO-243-211
- K1, K2, K3, K4, K5, K6, K7, K8: value HFE20-1-024-1HD504 -> HFE20-1/24-1HSD-L2
- R1: value 680 -> 680 500mW
Changed lines of the file:
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@@
 			)
 		)
-		(property "Value" "HFE20-1-024-1HD504"
+		(property "Value" "HFE20-1/24-1HSD-L2"
 			(at 7.52 4.475 0)
 			(layer "F.Fab")
@@
 		(tags "Diode Mini-MELF (SOD-80)")
 		(property "Reference" "D2"
-			(at 0 -2 360)
+			(at 0 -2 0)
 			(layer "F.SilkS")
 			(effects
@@
 		)
 		(property "Value" "12V"
-			(at 0 2 360)
+			(at 0 2 0)
 			(layer "F.Fab")
 			(effects
@@
 		)
 		(fp_text user "${REFERENCE}"
-			(at 0 -2 360)
+			(at 0 -2 0)
 			(layer "F.Fab")
 			(effects
@@
 			)
 		)
-		(property "Value" "HFE20-1-024-1HD504"
+		(property "Value" "HFE20-1/24-1HSD-L2"
 			(at 7.52 4.475 180)
 			(layer "F.Fab")
@@
 			)
 		)
-		(property "Value" "HFE20-1-024-1HD504"
+		(property "Value" "HFE20-1/24-1HSD-L2"
 			(at 7.52 4.475 180)
 			(layer "F.Fab")
@@
 			)
 		)
-		(property "Value" "HFE20-1-024-1HD504"
+		(property "Value" "HFE20-1/24-1HSD-L2"
 			(at 7.52 4.475 0)
 			(layer "F.Fab")
@@
 			)
 		)
-		(property "Value" "EIB_WAGO_243-211"
+		(property "Value" "WAGO-243-211"
 			(at 3.175 7.874 -90)
 			(layer "F.Fab")
@@
 			)
 		)
-		(property "Value" "HFE20-1-024-1HD504"
+		(property "Value" "HFE20-1/24-1HSD-L2"
 			(at 7.52 4.475 180)
 			(layer "F.Fab")
@@
 			)
 		)
-		(property "Value" "HFE20-1-024-1HD504"
+		(property "Value" "HFE20-1/24-1HSD-L2"
 			(at 7.52 4.475 180)
 			(layer "F.Fab")
@@
 			)
 		)
-		(property "Value" "HFE20-1-024-1HD504"
+		(property "Value" "HFE20-1/24-1HSD-L2"
 			(at 7.52 4.475 0)
 			(layer "F.Fab")
@@
 			)
 		)
-		(property "Value" "HFE20-1-024-1HD504"
+		(property "Value" "HFE20-1/24-1HSD-L2"
 			(at 7.52 4.475 0)
 			(layer "F.Fab")
@@
 			)
 		)
-		(property "Value" "680"
+		(property "Value" "680 500mW"
 			(at 0 -1.82 -90)
 			(layer "B.Fab")
