File: applications_din/in-out_2x-2x_2MU/2in-2out_2.0/2in-2out_2.0.kicad_pcb (KiCad board)
At the start: 2 copper layers, 86.5 x 33 mm, 62 parts, among them IC1 ULN2803, J1 Con_CTRL, J2 Con_IO, J3 Con_230V, K1 HFE20-1/24-1HSD-L2, K2 HFE20-1/24-1HSD-L2, U1 74HC595, U2 74HC165, X9 W237-102

Commit message: just all all projects for backup
Parts:
- removed J3: Con_230V, TerminalBlock_Phoenix:TerminalBlock_Phoenix_MKDS-3-6-5.08_1x06_P5.08mm_Horizontal
- added J5: Con_230V, selfbus:TerminalBlock_MetzConnect_Type701_RT11L03HGLU_1x04_P6.35mm_Horizontal, F.Cu at (111.4, 42.7)
- J2: footprint TerminalBlock_Phoenix:TerminalBlock_Phoenix_MKDS-1,5-4-5.08_1x04_P5.08mm_Horizontal -> TerminalBlock_Phoenix:TerminalBlock_Phoenix_PT-1,5-4-3.5-H_1x04_P3.50mm_Horizontal
- X9: footprint selfbus:W237-102 -> selfbus:W243-211_1x02_P5.75
- moved J2 10.5 mm to (186.3, 50.1), turned to 90 degrees
- moved X9 4.07 mm to (184.8, 65.4), turned to 90 degrees
- moved D1 1.65 mm to (177.8, 64.5), turned to 90 degrees
Connections:
- J2 pad 1: /IN1 -> /IO4
- J2 pad 2: /IN2 -> /IO3
- J2 pad 3: /IO3 -> /IN2
- J2 pad 4: /IO4 -> /IN1
Routing:
- net unconnected-(K2-Pad12): track 7.50 -> 0.00 mm
- net unconnected-(K1-Pad12): track 7.50 -> 0.00 mm
- net /HV_1B: track 21.0 -> 16.4 mm
- net /HV_2A: track 26.3 -> 24.2 mm
- net /HV_1A: track 22.9 -> 21.6 mm
- net /IO3: track 6.57 -> 7.84 mm
- net /IO4: track 7.10 -> 8.05 mm
- net /HV_2B: track 16.3 -> 16.8 mm
- added copper zone on F.Cu, net /HV_1A

Commit message: update
Parts:
- HUT_CNMB_2: renamed from REF**; value Val** -> BOT
- moved J5 0.90 mm to (112.3, 42.7)
Routing:
- net unconnected-(K2-Pad12): track 0.00 -> 7.50 mm
- net unconnected-(K1-Pad12): track 0.00 -> 7.50 mm
- net /HV_2A: track 24.2 -> 23.0 mm
- net /HV_1B: track 16.4 -> 15.5 mm
- net /HV_1A: track 21.6 -> 20.7 mm
Other:
- board text added: "- bus +"
- board text added: "www.selfbus.org Kombiaktor 4in 2out v2.0"
- board text removed: "-bus+"
- board text removed: "www.selfbus.org Kombiaktor 2in 2out v2.0"
Changed lines of the file:
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@@
 		(layer "F.Cu")
 		(at 193.562092 70.251281 90)
-		(property "Reference" "REF**"
-			(at 0.001281 1.187908 90)
+		(property "Reference" "HUT_CNMB_2"
+			(at 2.687281 1.763908 90)
 			(layer "F.SilkS")
 			(effects
@@
 			)
 		)
-		(property "Value" "Val**"
-			(at 0 2.937908 90)
+		(property "Value" "BOT"
+			(at 0 0 90)
 			(layer "F.Fab")
 			(effects
@@
 			(layer "F.SilkS")
 		)
-		(fp_circle
-			(center 28.5 -69.75)
-			(end 30.5 -69.75)
-			(stroke
-				(width 0.127)
-				(type solid)
-			)
-			(fill none)
-			(layer "F.SilkS")
-		)
-		(fp_circle
-			(center 7.5 -19.75)
-			(end 9.5 -19.75)
-			(stroke
-				(width 0.127)
-				(type solid)
-			)
-			(fill none)
-			(layer "F.SilkS")
-		)
 		(fp_line
 			(start 34.5 -88)
@@
 		)
 		(fp_circle
+			(center 28.5 -69.75)
+			(end 30.5 -69.75)
+			(stroke
+				(width 0.127)
+				(type solid)
+			)
+			(fill none)
+			(layer "F.Fab")
+		)
+		(fp_circle
+			(center 7.5 -19.75)
+			(end 9.5 -19.75)
+			(stroke
+				(width 0.127)
+				(type solid)
+			)
+			(fill none)
+			(layer "F.Fab")
+		)
+		(fp_circle
 			(center 30.7 -7.3)
 			(end 32.65 -7.3)
@@
 		)
 		(group ""
-			(members "306cf00c-0374-41ab-a57b-43949ed8a943" "3726c03a-e010-40e0-8791-36a4dd3362ae"
-				"72185549-7645-45dd-9e1b-01ed4b3f2402" "7ff5de72-f014-4ae4-abda-575f2f48d63d"
-				"9d9fca7a-6b73-4985-b8a2-5e18dfdd39b5" "c46f53d1-dd62-41bd-86ce-a87c65a1f4fb"
+			(members "21b02721-2c10-4749-b1ce-93345cff606c" "623aa02e-4e70-4b69-9cfb-99e1a25f2398"
+				"81b68e20-831f-465e-a050-1e0d30abec21" "a68db552-db5c-428b-bdef-248c72037c54"
+				"bc136528-94da-4a8d-add4-f4ba8c316f03" "f7e6d3e1-a216-4e12-8875-2223dc941314"
 			)
 		)
 		(group ""
-			(members "082181ad-8bd1-482f-9b92-210d3a7a287d" "13881293-000b-4ca1-8b7d-4781b717b719"
-				"28f5213b-c144-490d-94a5-66a9139aee38" "679cebbf-7ea2-4739-94fa-5cade1d61a0c"
-				"d61cf254-5cae-45ab-8527-669c51b9ed63" "f91a2f59-9010-42b8-91a3-6454608b9996"
+			(members "00f021b2-411b-474a-aff4-2e844cdc37df" "085059c5-68c3-42f0-9523-040ace970e91"
+				"5d8287bc-8f49-4156-89de-17f0b19e46bf" "7706722f-4874-44a3-8322-643fa3909165"
+				"a320a89c-b2ef-4f5c-adf5-99b48c7cac22" "add3b6a5-4888-440c-a2a4-995673f5d78b"
 			)
 		)
@@
 		)
 		(property "Value" "W237-102"
-			(at 3.175 7.874 270)
+			(at 3.175 7.874 -90)
 			(layer "F.Fab")
 			(effects
@@
 		)
 		(fp_text user "${REFERENCE}"
-			(at 3.175 3.175 270)
+			(at 3.175 3.175 -90)
 			(layer "F.Fab")
 			(effects
@@
 		(tags "Diode SMA (DO-214AC)")
 		(property "Reference" "D1"
-			(at 4.445 0 360)
+			(at 4.445 0 0)
 			(layer "F.SilkS")
 			(effects
@@
 		)
 		(property "Value" "SMAJ40CA"
-			(at 0 2.6 270)
+			(at 0 2.6 -90)
 			(layer "F.Fab")
 			(effects
@@
 		)
 		(fp_text user "${REFERENCE}"
-			(at 0 -2.5 270)
+			(at 0 -2.5 -90)
 			(layer "F.Fab")
 			(effects
@@
 		)
 		(property "Value" "Con_IO"
-			(at 5.25 5.56 270)
+			(at 5.25 5.56 -90)
 			(layer "F.Fab")
 			(effects
@@
 		(tags "test point SMD pad")
 		(property "Reference" "TP3"
-			(at 1.988 0 90)
+			(at 2.242 0 90)
 			(layer "F.SilkS")
 			(effects
@@
 	(footprint "selfbus:TerminalBlock_MetzConnect_Type701_RT11L03HGLU_1x04_P6.35mm_Horizontal"
 		(layer "F.Cu")
-		(at 111.366051 42.727996 -90)
+		(at 112.268 42.727996 -90)
 		(descr "terminal block Metz Connect Type701_RT11L03HGLU, 3 pins, pitch 6.35mm, size 19x12.5mm^2, drill diamater 1.3mm, pad diameter 2.5mm, see http://www.metz-connect.com/de/system/files/productfiles/Datenblatt_317011_RT11LxxHGLU_OFF-022798U.pdf, script-generated using https://github.com/pointhi/kicad-footprint-generator/scripts/TerminalBlock_MetzConnect")
 		(tags "THT terminal block Metz Connect Type701_RT11L03HGLU pitch 6.35mm size 19x12.5mm^2 drill 1.3mm pad 2.5mm")
 		(property "Reference" "J5"
-			(at 10.3124 -5.6896 -90)
+			(at -4.373996 0 0)
 			(layer "F.SilkS")
 			(effects
@@
 	)
 	(gr_line
-		(start 114.046 59.944)
-		(end 114.046 61.468)
+		(start 133.477 57.785)
+		(end 133.477 59.309)
 		(stroke
 			(width 0.3048)
@@
 	)
 	(gr_line
-		(start 114.046 61.468)
-		(end 114.808 62.992)
+		(start 133.477 59.309)
+		(end 134.239 60.833)
 		(stroke
 			(width 0.3048)
@@
 	)
 	(gr_line
-		(start 114.046 42.672)
-		(end 114.046 44.704)
+		(start 133.731 44.323)
+		(end 133.731 46.355)
 		(stroke
 			(width 0.3048)
@@
 	)
 	(gr_line
-		(start 114.046 44.704)
-		(end 113.03 44.704)
+		(start 133.731 46.355)
+		(end 132.715 46.355)
 		(stroke
 			(width 0.3048)
@@
 	)
 	(gr_line
-		(start 113.03 39.624)
-		(end 114.046 39.624)
+		(start 132.715 41.275)
+		(end 133.731 41.275)
 		(stroke
 			(width 0.3048)
@@
 	)
 	(gr_line
-		(start 113.03 59.944)
-		(end 114.046 59.944)
+		(start 132.461 57.785)
+		(end 133.477 57.785)
 		(stroke
 			(width 0.3048)
@@
 	)
 	(gr_line
-		(start 114.046 62.992)
-		(end 114.046 65.024)
+		(start 133.477 60.833)
+		(end 133.477 62.865)
 		(stroke
 			(width 0.3048)
@@
 	)
 	(gr_line
-		(start 114.046 65.024)
-		(end 113.03 65.024)
+		(start 133.477 62.865)
+		(end 132.461 62.865)
 		(stroke
 			(width 0.3048)
@@
 	)
 	(gr_line
-		(start 114.046 41.148)
-		(end 114.808 42.672)
+		(start 133.731 42.799)
+		(end 134.493 44.323)
 		(stroke
 			(width 0.3048)
@@
 	)
 	(gr_line
-		(start 114.046 39.624)
-		(end 114.046 41.148)
+		(start 133.731 41.275)
+		(end 133.731 42.799)
 		(stroke
 			(width 0.3048)
@@
 	)
 	(gr_text "K1"
-		(at 117.221 40.513 -90)
+		(at 136.906 42.164 -90)
 		(layer "B.SilkS")
 		(effects
@@
 	)
 	(gr_text "K2"
-		(at 117.094 60.706 -90)
+		(at 136.525 58.547 -90)
 		(layer "B.SilkS")
 		(effects
@@
 		)
 	)
-	(gr_text "-bus+"
-		(at 181.0004 62.5856 -90)
+	(gr_text "- bus +"
+		(at 189.145 62.738 270)
 		(layer "B.SilkS")
 		(effects
@@
 		)
 	)
-	(gr_text "www.selfbus.org\nKombiaktor\n2in 2out v2.0"
+	(gr_text "www.selfbus.org\nKombiaktor\n4in 2out v2.0"
 		(at 153.416 47.75 0)
 		(layer "F.SilkS")
@@
 	)
 	(segment
-		(start 113.594047 40.5)
+		(start 112.268 42.727996)
+		(end 112.268 41.826047)
+		(width 2.4)
+		(layer "B.Cu")
+		(net 31)
+	)
+	(segment
+		(start 119.75 48)
 		(end 119.75 40.5)
 		(width 2.4)
@@
 	)
 	(segment
-		(start 111.366051 42.727996)
+		(start 112.268 41.826047)
 		(end 113.594047 40.5)
 		(width 2.4)
@@
 	)
 	(segment
-		(start 119.75 48)
+		(start 113.594047 40.5)
 		(end 119.75 40.5)
 		(width 2.4)
@@
 	)
 	(segment
-		(start 116.532 44.25)
-		(end 118 44.25)
+		(start 112.268 49.077996)
+		(end 113.736004 49.077996)
 		(width 2.4)
 		(layer "F.Cu")
@@
 	)
 	(segment
-		(start 111.366051 49.077996)
-		(end 113.736004 49.077996)
+		(start 124.79 44.5)
+		(end 124.79 48)
 		(width 2.4)
 		(layer "F.Cu")
@@
 	)
 	(segment
-		(start 124.79 44.5)
-		(end 124.79 48)
+		(start 113.736004 49.077996)
+		(end 115.062 47.752)
 		(width 2.4)
 		(layer "F.Cu")
@@
 	)
 	(segment
-		(start 113.736004 49.077996)
-		(end 115.57 47.244)
+		(start 115.062 46.228)
+		(end 117.04 44.25)
 		(width 2.4)
 		(layer "F.Cu")
@@
 	)
 	(segment
-		(start 115.57 45.212)
-		(end 116.532 44.25)
+		(start 124.79 40.5)
+		(end 124.79 44.5)
 		(width 2.4)
 		(layer "F.Cu")
@@
 	)
 	(segment
-		(start 124.79 40.5)
-		(end 124.79 44.5)
+		(start 117.04 44.25)
+		(end 118 44.25)
 		(width 2.4)
 		(layer "F.Cu")
@@
 	)
 	(segment
-		(start 115.57 47.244)
-		(end 115.57 45.212)
+		(start 124.54 44.25)
+		(end 124.79 44.5)
 		(width 2.4)
 		(layer "F.Cu")
@@
 	)
 	(segment
-		(start 124.54 44.25)
-		(end 124.79 44.5)
+		(start 115.062 47.752)
+		(end 115.062 46.228)
 		(width 2.4)
 		(layer "F.Cu")
@@
 	)
 	(segment
-		(start 119.75 56.75)
-		(end 118.427996 55.427996)
+		(start 118.427996 55.427996)
+		(end 112.268 55.427996)
 		(width 2.4)
 		(layer "B.Cu")
@@
 	)
 	(segment
-		(start 118.427996 55.427996)
-		(end 111.366051 55.427996)
+		(start 119.75 56.75)
+		(end 118.427996 55.427996)
 		(width 2.4)
 		(layer "B.Cu")
@@
 	)
 	(segment
-		(start 111.359754 61.784293)
-		(end 112.644047 60.5)
+		(start 112.261703 61.784293)
+		(end 113.545996 60.5)
 		(width 2.4)
 		(layer "F.Cu")
@@
 	)
 	(segment
-		(start 124.79 56.75)
-		(end 124.79 60.75)
+		(start 113.545996 60.5)
+		(end 118 60.5)
 		(width 2.4)
 		(layer "F.Cu")
@@
 	)
 	(segment
-		(start 112.644047 60.5)
-		(end 118 60.5)
+		(start 124.79 56.75)
+		(end 124.79 60.75)
 		(width 2.4)
 		(layer "F.Cu")
@@
 		(net 55)
 	)
+	(segment
+		(start 129.83 56.75)
+		(end 129.83 64.25)
+		(width 2.4)
+		(layer "F.Cu")
+		(net 56)
+	)
+	(segment
+		(start 129.83 40.5)
+		(end 129.83 48)
+		(width 2.4)
+		(layer "F.Cu")
+		(net 57)
+	)
 	(zone
 		(net 32)
@@
 		(polygon
 			(pts
-				(xy 109.474 51.054) (xy 109.492 46.736) (xy 113.284 46.736) (xy 113.284 45.212) (xy 116.84 45.212)
-				(xy 116.84 51.054)
+				(xy 109.474 51.054) (xy 109.492 45.974) (xy 116.84 45.974) (xy 116.84 51.054)
 			)
 		)
@@
 		(polygon
 			(pts
-				(xy 117.094 59.182) (xy 117.076 61.976) (xy 114.3 61.976) (xy 114.3 64.516) (xy 109.22 64.516) (xy 109.22 59.182)
+				(xy 117.094 59.182) (xy 117.076 61.976) (xy 115.316 61.976) (xy 115.316 64.516) (xy 109.22 64.516)
+				(xy 109.22 59.182)
 			)
 		)
@@
 		(polygon
 			(pts
-				(xy 109.492 54.246) (xy 121.412 54.246) (xy 121.412 66.548) (xy 116.586 66.548) (xy 116.586 58.42)
-				(xy 115.316 57.436) (xy 109.492 57.436)
+				(xy 109.492 53.484) (xy 121.666 53.484) (xy 121.666 66.548) (xy 116.586 66.548) (xy 116.586 58.928)
+				(xy 114.808 57.436) (xy 109.492 57.436)
 			)
 		)

Commit message: update in-out_4x-2x_2MU - final for now
Parts:
- removed X9: W237-102, selfbus:W243-211_1x02_P5.75
- added J4: EIB_WAGO_243-211, selfbus:W243-211_1x02_P5.75, F.Cu at (184.7, 65.4)
Routing:
- net unconnected-(K2-Pad12): track 7.50 -> 0.00 mm
- net unconnected-(K1-Pad12): track 7.50 -> 0.00 mm
Other:
- board text added: "www.selfbus.org Kombiaktor 4in 2out v1.0"
- board text removed: "www.selfbus.org Kombiaktor 4in 2out v2.0"

Commit message: update all stuff
Parts:
- J1: footprint Connector_PinHeader_2.54mm:PinHeader_1x09_P2.54mm_Vertical -> Connector_Molex:Molex_KK-254_AE-6410-10A_1x10_P2.54mm_Vertical
- U2: renamed from IC1; value ULN2803 -> ULN2803A
- moved TP7 2.29 mm to (173.2, 59.6)
- moved R1 2.13 mm to (170.2, 60.2)
- moved TP9 1.99 mm to (152.1, 61.3)
- moved SJ1 1.88 mm to (167.4, 60.7)
- moved TP8 1.50 mm to (157.4, 61.3)
- moved TP3 1.41 mm to (160.0, 61.3)
- moved TP1 1.40 mm to (149.5, 61.3)
- moved C1 0.38 mm to (162.9, 57.8)
- moved J1 0.15 mm to (149.6, 66.0), turned to 0 degrees
- renumbered U2 to U3
Connections:
- J1 pad 1: VBUS -> GND
- J1 pad 2: GND -> VBUS
- J1 pad 3: +3V3 -> GND
- J1 pad 4: /PWM -> +3V3
- J1 pad 5: /MOSI -> /PWM
- J1 pad 6: /SSEL -> /MOSI
- J1 pad 7: /MISO -> /SSEL
- J1 pad 8: /SCK -> /MISO
- J1 pad 9: /EIB_DC -> /SCK
Routing:
- net /PWM: track 3.42 -> 5.70 mm
- net VDD: track 77.9 -> 79.8 mm
- net /SCK: track 45.7 -> 47.5 mm
- net +3V3: track 102.5 -> 101.3 mm, vias 6 -> 7
- net /MISO: track 30.9 -> 32.1 mm
- net /SSEL: track 42.1 -> 43.2 mm
- net /EIB_DC: track 11.1 -> 12.2 mm
- net GND: track 1.78 -> 2.81 mm
- net /MOSI: track 24.8 -> 25.8 mm
- net VBUS: track 43.0 -> 43.7 mm

Commit message: finally standardize selected parts on all boards
Parts:
- J4: value EIB_WAGO_243-211 -> WAGO-243-211
Changed lines of the file:
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@@
 			)
 		)
-		(property "Value" "EIB_WAGO_243-211"
+		(property "Value" "WAGO-243-211"
 			(at 3.175 7.874 -90)
 			(layer "F.Fab")

Commit message: final for manufacturing
Parts:
- J2: footprint TerminalBlock_Phoenix:TerminalBlock_Phoenix_PT-1,5-4-3.5-H_1x04_P3.50mm_Horizontal -> TerminalBlock_Phoenix:TerminalBlock_Phoenix_PTSM-0,5-4-2.5-H-THR_1x04_P2.50mm_Horizontal
- R1: value 680 -> 680 500mW
- moved C4 3.45 mm to (180.2, 44.2), turned to 0 degrees
- moved J2 3.07 mm to (188.9, 48.5)
- moved D2 1.02 mm to (177.0, 41.9)
- moved TVS1 0.76 mm to (178.3, 47.1)
- moved F2 0.18 mm to (179.3, 46.2)
- moved FB2 0.17 mm to (179.2, 44.3)
- moved TP11 0.05 mm to (180.0, 48.3)
Routing:
- net /IO4: track 8.05 -> 12.8 mm
- net /IO3: track 7.84 -> 12.0 mm
- net /IN1: track 7.33 -> 11.0 mm
- net /IN2: track 6.37 -> 8.99 mm
- net +3V3: track 101.3 -> 102.2 mm
- net /IN4: track 18.6 -> 17.9 mm
- net GND: vias 13 -> 17

Commit message: update in-out_4x-2x_2MU
Parts:
- R1: value 680 500mW -> 470 500mW
Changed lines of the file:
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@@
 	(net 54 "unconnected-(K1-Pad12)")
 	(net 55 "unconnected-(K2-Pad12)")
-	(net 56 "unconnected-(K1-Pad12)_0")
-	(net 57 "unconnected-(K2-Pad12)_0")
+	(net 56 "unconnected-(K1-Pad12)_1")
+	(net 57 "unconnected-(K2-Pad12)_1")
 	(net 58 "Net-(TVS1-I{slash}O2)")
 	(net 59 "Net-(TVS1-I{slash}O3)")
@@
 			(layers "*.Cu" "*.Mask")
 			(remove_unused_layers no)
-			(net 57 "unconnected-(K2-Pad12)_0")
+			(net 57 "unconnected-(K2-Pad12)_1")
 			(pintype "passive+no_connect")
 			(solder_mask_margin 0.0508)
@@
 		(sheetname "Stammblatt")
 		(sheetfile "4in-2out_1.0.kicad_sch")
-		(attr exclude_from_pos_files)
+		(attr exclude_from_pos_files exclude_from_bom)
 		(fp_circle
 			(center 0 0)
@@
 		(sheetname "Stammblatt")
 		(sheetfile "4in-2out_1.0.kicad_sch")
-		(attr smd)
+		(attr smd dnp)
 		(fp_line
 			(start 1.75 -1.11)
@@
 		(sheetname "Stammblatt")
 		(sheetfile "4in-2out_1.0.kicad_sch")
-		(attr exclude_from_pos_files)
+		(attr exclude_from_pos_files exclude_from_bom)
 		(fp_circle
 			(center 0 0)
@@
 		(sheetname "Stammblatt")
 		(sheetfile "4in-2out_1.0.kicad_sch")
-		(attr exclude_from_pos_files)
+		(attr exclude_from_pos_files exclude_from_bom)
 		(fp_circle
 			(center 0 0)
@@
 		(sheetname "Stammblatt")
 		(sheetfile "4in-2out_1.0.kicad_sch")
-		(attr exclude_from_pos_files)
+		(attr exclude_from_pos_files exclude_from_bom)
 		(fp_circle
 			(center 0 0)
@@
 		(sheetname "Stammblatt")
 		(sheetfile "4in-2out_1.0.kicad_sch")
-		(attr exclude_from_pos_files)
+		(attr exclude_from_pos_files exclude_from_bom)
 		(fp_circle
 			(center 0 0)
@@
 			(layers "*.Cu" "*.Mask")
 			(remove_unused_layers no)
-			(net 56 "unconnected-(K1-Pad12)_0")
+			(net 56 "unconnected-(K1-Pad12)_1")
 			(pintype "passive+no_connect")
 			(solder_mask_margin 0.0508)
@@
 		(sheetfile "4in-2out_1.0.kicad_sch")
 		(zone_connect 1)
-		(attr exclude_from_pos_files)
+		(attr exclude_from_pos_files exclude_from_bom)
 		(fp_line
 			(start 1.4 -1)
@@
 		(sheetname "Stammblatt")
 		(sheetfile "4in-2out_1.0.kicad_sch")
-		(attr exclude_from_pos_files)
+		(attr exclude_from_pos_files exclude_from_bom)
 		(fp_circle
 			(center 0 0)
@@
 		(sheetname "Stammblatt")
 		(sheetfile "4in-2out_1.0.kicad_sch")
-		(attr exclude_from_pos_files)
+		(attr exclude_from_pos_files exclude_from_bom)
 		(fp_circle
 			(center 0 0)
@@
 		(sheetname "Stammblatt")
 		(sheetfile "4in-2out_1.0.kicad_sch")
-		(attr exclude_from_pos_files)
+		(attr exclude_from_pos_files exclude_from_bom)
 		(fp_circle
 			(center 0 0)
@@
 			)
 		)
-		(property "Value" "680 500mW"
+		(property "Value" "470 500mW"
 			(at 0 1.82 90)
 			(layer "F.Fab")
@@
 		(sheetname "Stammblatt")
 		(sheetfile "4in-2out_1.0.kicad_sch")
-		(attr exclude_from_pos_files)
+		(attr exclude_from_pos_files exclude_from_bom)
 		(fp_circle
 			(center 0 0)
@@
 		(sheetname "Stammblatt")
 		(sheetfile "4in-2out_1.0.kicad_sch")
-		(attr exclude_from_pos_files)
+		(attr exclude_from_pos_files exclude_from_bom)
 		(fp_circle
 			(center 0 0)
@@
 		(sheetname "Stammblatt")
 		(sheetfile "4in-2out_1.0.kicad_sch")
-		(attr exclude_from_pos_files)
+		(attr exclude_from_pos_files exclude_from_bom)
 		(fp_circle
 			(center 0 0)
@@
 		(sheetname "Stammblatt")
 		(sheetfile "4in-2out_1.0.kicad_sch")
-		(attr exclude_from_pos_files)
+		(attr exclude_from_pos_files exclude_from_bom)
 		(fp_circle
 			(center 0 0)
@@
 		(sheetname "Stammblatt")
 		(sheetfile "4in-2out_1.0.kicad_sch")
-		(attr exclude_from_pos_files)
+		(attr exclude_from_pos_files exclude_from_bom)
 		(fp_circle
 			(center 0 0)
@@
 		(sheetfile "4in-2out_1.0.kicad_sch")
 		(zone_connect 1)
-		(attr exclude_from_pos_files)
+		(attr exclude_from_pos_files exclude_from_bom)
 		(fp_line
 			(start 1.4 -1)
@@
 		(sheetfile "4in-2out_1.0.kicad_sch")
 		(zone_connect 1)
-		(attr exclude_from_pos_files)
+		(attr exclude_from_pos_files exclude_from_bom)
 		(fp_line
 			(start 1.4 -1)
@@
 		(sheetfile "4in-2out_1.0.kicad_sch")
 		(zone_connect 1)
-		(attr exclude_from_pos_files)
+		(attr exclude_from_pos_files exclude_from_bom)
 		(fp_line
 			(start -1.4 1)
@@
 		(tags "capacitor")
 		(property "Reference" "C4"
-			(at -2.667 0 360)
+			(at -2.667 0 0)
 			(layer "B.SilkS")
 			(effects
@@
 		)
 		(property "Value" "100n"
-			(at 0 -1.68 360)
+			(at 0 -1.68 0)
 			(layer "B.Fab")
 			(effects
@@
 		)
 		(fp_text user "${REFERENCE}"
-			(at 0 0.225 360)
+			(at 0 0.225 0)
 			(layer "B.Fab")
 			(effects
@@
 		(sheetfile "4in-2out_1.0.kicad_sch")
 		(zone_connect 1)
-		(attr exclude_from_pos_files)
+		(attr exclude_from_pos_files exclude_from_bom)
 		(fp_line
 			(start -1.4 1)
@@
 		(sheetfile "4in-2out_1.0.kicad_sch")
 		(zone_connect 1)
-		(attr exclude_from_pos_files)
+		(attr exclude_from_pos_files exclude_from_bom)
 		(fp_line
 			(start -1.4 1)
@@
 		(sheetfile "4in-2out_1.0.kicad_sch")
 		(zone_connect 1)
-		(attr exclude_from_pos_files)
+		(attr exclude_from_pos_files exclude_from_bom)
 		(fp_line
 			(start 1.4 -1)
