File: applications_din/in-out_2x-2x_2MU/2in-2out_2.0/2in-2out_2.0.kicad_sch (KiCad schematic)
At the start: 62 parts, among them IC1 ULN2803, J1 Con_CTRL, J2 Con_IO, J3 Con_230V, J4 Con_EIB_WAGO_243-211, K1 HFE20-1/24-1HSD-L2, K2 HFE20-1/24-1HSD-L2, U1 74HC595, U2 74HC165, X9 W237-102

Commit message: just all all projects for backup
Parts:
- added J5: Con_230V, selfbus:TerminalBlock_MetzConnect_Type701_RT11L03HGLU_1x04_P6.35mm_Horizontal, symbol Connector:Conn_01x04_Socket
- J2: footprint TerminalBlock_Phoenix:TerminalBlock_Phoenix_MKDS-1,5-4-5.08_1x04_P5.08mm_Horizontal -> TerminalBlock_Phoenix:TerminalBlock_Phoenix_PT-1,5-4-3.5-H_1x04_P3.50mm_Horizontal
- J3: now not fitted
- X9: footprint selfbus:W237-102 -> selfbus:W243-211_1x02_P5.75
Connections:
- net HV_1A: now also J5.4 (Pin_4)
- net HV_1B: now also J5.3 (Pin_3)
- net HV_2A: now also J5.2 (Pin_2)
- net HV_2B: now also J5.1 (Pin_1)
- net IN1: now also J2.4 (Pin_4); no longer J2.1 (Pin_1)
- net IN2: now also J2.3 (Pin_3); no longer J2.2 (Pin_2)
- net IO3: now also J2.2 (Pin_2); no longer J2.3 (Pin_3)
- net IO4: now also J2.1 (Pin_1); no longer J2.4 (Pin_4)

Commit message: update in-out_4x-2x_2MU - final for now
Parts:
- removed X9: W237-102, selfbus:W243-211_1x02_P5.75, symbol selfbus:W237-102
- J4: value Con_EIB_WAGO_243-211 -> EIB_WAGO_243-211; footprint (none) -> selfbus:W243-211_1x02_P5.75
Connections:
- net GND: now also J4.1 (Pin_1); no longer J4.2 (Pin_2)
- net VBUS: now also J4.2 (Pin_2); no longer J4.1 (Pin_1)
Other:
- note added: "1.0"
- note added: "2-fach Binärausgang 230V 16A + 2- bis 4-fach Binäreingang (ARM): -R1 bestücken -SJ1 nicht brücken -für C1 220µF/63V verwenden -C2 nicht bestücken -24V Relais (HFE20-1/24-XXXD-L2...) verwenden (ggf. alternativ Omron G5RL-K1A-EL-HA DC24, leider single coil) (ggf. alternativ Finder 41.61.6.012.4016, bei Reichelt nur 12V und kein high inrush)"
- note added: "4in-2out 16A Application Board"
- note removed: "2-fach Binärausgang 230V 16A + 2-fach Binäreingang (ARM): -R1 bestücken -SJ1 nicht brücken -für C1 220µF/63V verwenden -C2 nicht bestücken -24V Relais (HFE20-1/24-XXXD-L2...) verwenden (ggf. alternativ Omron G5RL-K1A-EL-HA DC24, leider single coil) (ggf. alternativ Finder 41.61.6.012.4016, bei Reichelt nur 12V und kein high inrush)"
- note removed: "2.0"
- note removed: "2in-2out 16A Application Board"
- moved on the sheet: C4, J4

Commit message: update all stuff
Parts:
- J1: footprint Connector_PinHeader_2.54mm:PinHeader_1x09_P2.54mm_Vertical -> Connector_Molex:Molex_KK-254_AE-6410-10A_1x10_P2.54mm_Vertical; symbol Connector:Conn_01x09_Socket -> Connector_Generic:Conn_01x10
- J4: symbol Connector:Conn_01x02_Socket -> Connector:Screw_Terminal_01x02
- U2: renamed from IC1; value ULN2803 -> ULN2803A
- renumbered U2 to U3
Connections:
- net +3V3: now also J1.4 (Pin_4); no longer J1.3 (Pin_3)
- net EIB_DC: now also J1.10 (Pin_10); no longer J1.9 (Pin_9)
- net GND: now also J1.1 (Pin_1), J1.3 (Pin_3); no longer J1.2 (Pin_2)
- net MISO: now also J1.8 (Pin_8); no longer J1.7 (Pin_7)
- net MOSI: now also J1.6 (Pin_6); no longer J1.5 (Pin_5)
- net PWM: now also J1.5 (Pin_5); no longer J1.4 (Pin_4)
- net SCK: now also J1.9 (Pin_9); no longer J1.8 (Pin_8)
- net SSEL: now also J1.7 (Pin_7); no longer J1.6 (Pin_6)
- net VBUS: now also J1.2 (Pin_2); no longer J1.1 (Pin_1)
- no-connect marks 10 -> 9
Other:
- moved on the sheet: J5
Changed lines of the file:
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@@
 	)
 	(junction
+		(at 40.64 35.56)
+		(diameter 0)
+		(color 0 0 0 0)
+	)
+	(junction
 		(at 203.2 38.1)
 		(diameter 0)
@@
 	)
 	(no_connect
-		(at 109.22 175.26)
-	)
-	(no_connect
 		(at 60.96 190.5)
 	)
@@
 	(wire
 		(pts
+			(xy 33.02 35.56) (xy 40.64 35.56)
+		)
+		(stroke
+			(width 0)
+			(type default)
+		)
+	)
+	(wire
+		(pts
 			(xy 35.56 167.64) (xy 40.64 167.64)
 		)
@@
 	(wire
 		(pts
-			(xy 35.56 40.64) (xy 33.02 40.64)
+			(xy 33.02 40.64) (xy 40.64 40.64)
 		)
 		(stroke
@@
 	(wire
 		(pts
+			(xy 40.64 40.64) (xy 40.64 35.56)
+		)
+		(stroke
+			(width 0)
+			(type default)
+		)
+	)
+	(wire
+		(pts
 			(xy 132.08 121.92) (xy 137.16 121.92)
 		)
@@
 	)
 	(label "HV_2B"
-		(at 189.865 173.355 180)
+		(at 190.5 173.99 180)
 		(fields_autoplaced yes)
 		(effects
@@
 		)
 	)
+	(label "O[1..8]"
+		(at 64.77 190.5 0)
+		(fields_autoplaced yes)
+		(effects
+			(font
+				(size 1.27 1.27)
+			)
+			(justify left bottom)
+		)
+	)
 	(label "IO4"
 		(at 269.24 60.96 0)
@@
 	)
 	(label "HV_1A"
-		(at 189.865 180.975 180)
+		(at 190.5 181.61 180)
 		(fields_autoplaced yes)
 		(effects
@@
 	)
 	(label "HV_1B"
-		(at 189.865 178.435 180)
+		(at 190.5 179.07 180)
 		(fields_autoplaced yes)
 		(effects
@@
 	)
 	(label "HV_2A"
-		(at 189.865 175.895 180)
+		(at 190.5 176.53 180)
 		(fields_autoplaced yes)
 		(effects
@@
 		(dnp no)
 		(fields_autoplaced yes)
-		(property "Reference" "U2"
-			(at 94.3259 36.4957 0)
+		(property "Reference" "U3"
+			(at 96.9965 36.4955 0)
 			(effects
 				(font
@@
 		)
 		(property "Value" "74HC165"
-			(at 94.3259 38.9199 0)
+			(at 96.9965 38.9198 0)
 			(effects
 				(font
@@
 			(project "4in-2out_1.0"
 				(path "/e17a8f7c-290a-48c4-8119-0faa75a2ce74"
-					(reference "U2")
+					(reference "U3")
 					(unit 1)
 				)
@@
 		(dnp no)
 		(fields_autoplaced yes)
-		(property "Reference" "IC1"
+		(property "Reference" "U2"
 			(at 86.36 157.3654 0)
 			(effects
@@
 			)
 		)
-		(property "Value" "ULN2803"
+		(property "Value" "ULN2803A"
 			(at 86.36 160.4898 0)
 			(effects
@@
 			(project "4in-2out_1.0"
 				(path "/e17a8f7c-290a-48c4-8119-0faa75a2ce74"
-					(reference "IC1")
+					(reference "U2")
 					(unit 1)
 				)
@@
 	(symbol
 		(lib_id "Connector:Conn_01x04_Socket")
-		(at 194.945 175.895 0)
+		(at 195.58 176.53 0)
 		(unit 1)
 		(exclude_from_sim no)
@@
 		(dnp no)
 		(property "Reference" "J5"
-			(at 195.6562 175.9528 0)
+			(at 196.2912 176.5878 0)
 			(effects
 				(font
@@
 		)
 		(property "Value" "Con_230V"
-			(at 195.6562 178.3771 0)
+			(at 196.2912 179.0121 0)
 			(effects
 				(font
@@
 		)
 		(property "Footprint" "selfbus:TerminalBlock_MetzConnect_Type701_RT11L03HGLU_1x04_P6.35mm_Horizontal"
-			(at 194.945 175.895 0)
+			(at 195.58 176.53 0)
 			(effects
 				(font
@@
 		)
 		(property "Datasheet" "~"
-			(at 194.945 175.895 0)
+			(at 195.58 176.53 0)
 			(effects
 				(font
@@
 		)
 		(property "Description" "Generic connector, single row, 01x04, script generated"
-			(at 194.945 175.895 0)
+			(at 195.58 176.53 0)
 			(effects
 				(font
@@
 		(pin "11"
 		)
-		(pin "11A"
-		)
-		(pin "14B"
-		)
 		(pin "12"
 		)
@@
 	(symbol
 		(lib_id "power:GND")
-		(at 35.56 40.64 90)
-		(unit 1)
-		(exclude_from_sim no)
-		(in_bom yes)
-		(on_board yes)
-		(dnp no)
-		(fields_autoplaced yes)
-		(property "Reference" "#PWR07"
-			(at 41.91 40.64 0)
-			(effects
-				(font
-					(size 1.27 1.27)
-				)
-				(hide yes)
-			)
-		)
-		(property "Value" "GND"
-			(at 38.735 40.64 90)
-			(effects
-				(font
-					(size 1.27 1.27)
-				)
-				(justify right)
-			)
-		)
-		(property "Footprint" ""
-			(at 35.56 40.64 0)
-			(effects
-				(font
-					(size 1.27 1.27)
-				)
-				(hide yes)
-			)
-		)
-		(property "Datasheet" ""
-			(at 35.56 40.64 0)
-			(effects
-				(font
-					(size 1.27 1.27)
-				)
-				(hide yes)
-			)
-		)
-		(property "Description" "Power symbol creates a global label with name \"GND\" , ground"
-			(at 35.56 40.64 0)
-			(effects
-				(font
-					(size 1.27 1.27)
-				)
-				(hide yes)
-			)
-		)
-		(pin "1"
-		)
-		(instances
-			(project "4in-2out_1.0"
-				(path "/e17a8f7c-290a-48c4-8119-0faa75a2ce74"
-					(reference "#PWR07")
-					(unit 1)
-				)
-			)
-		)
-	)
-	(symbol
-		(lib_id "power:GND")
 		(at 182.88 20.32 0)
 		(unit 1)
@@
 	)
 	(symbol
-		(lib_id "Connector:Conn_01x09_Socket")
-		(at 27.94 48.26 0)
+		(lib_id "Connector_Generic:Conn_01x10")
+		(at 27.94 45.72 0)
 		(mirror y)
 		(unit 1)
@@
 		(fields_autoplaced yes)
 		(property "Reference" "J1"
-			(at 28.575 33.4985 0)
+			(at 27.94 30.1455 0)
 			(effects
 				(font
@@
 		)
 		(property "Value" "Con_CTRL"
-			(at 28.575 35.9227 0)
+			(at 27.94 32.5698 0)
 			(effects
 				(font
@@
 			)
 		)
-		(property "Footprint" "Connector_PinHeader_2.54mm:PinHeader_1x09_P2.54mm_Vertical"
-			(at 27.94 48.26 0)
+		(property "Footprint" "Connector_Molex:Molex_KK-254_AE-6410-10A_1x10_P2.54mm_Vertical"
+			(at 27.94 45.72 0)
 			(effects
 				(font
@@
 		)
 		(property "Datasheet" "~"
-			(at 27.94 48.26 0)
+			(at 27.94 45.72 0)
 			(effects
 				(font
@@
 			)
 		)
-		(property "Description" "Generic connector, single row, 01x09, script generated"
-			(at 27.94 48.26 0)
+		(property "Description" "Generic connector, single row, 01x10, script generated (kicad-library-utils/schlib/autogen/connector/)"
+			(at 27.94 45.72 0)
 			(effects
 				(font
@@
 		(pin "8"
 		)
+		(pin "10"
+		)
 		(instances
 			(project "4in-2out_1.0"
@@
 		(fields_autoplaced yes)
 		(property "Reference" "U1"
-			(at 52.9941 160.9557 0)
+			(at 52.9941 160.9555 0)
 			(effects
 				(font
@@
 		)
 		(property "Value" "74HC595"
-			(at 52.9941 163.3799 0)
+			(at 52.9941 163.3798 0)
 			(effects
 				(font
@@
 	)
 	(symbol
-		(lib_id "Connector:Conn_01x02_Socket")
+		(lib_id "Connector:Screw_Terminal_01x02")
 		(at 25.4 109.22 180)
 		(unit 1)
@@
 		(fields_autoplaced yes)
 		(property "Reference" "J4"
-			(at 24.6889 106.7378 0)
+			(at 23.3681 106.7378 0)
 			(effects
 				(font
@@
 		)
 		(property "Value" "EIB_WAGO_243-211"
-			(at 24.6889 109.1621 0)
+			(at 23.3681 109.1621 0)
 			(effects
 				(font
@@
 			)
 		)
-		(property "Description" "Generic connector, single row, 01x02, script generated"
+		(property "Description" "Generic screw terminal, single row, 01x02, script generated (kicad-library-utils/schlib/autogen/connector/)"
 			(at 25.4 109.22 0)
 			(effects
@@
 		)
 		(property "Value" "VBUS"
-			(at 36.83 35.7449 90)
+			(at 36.83 34.29 90)
 			(effects
 				(font
@@
 		(pin "11"
 		)
-		(pin "11A"
-		)
-		(pin "14B"
-		)
 		(pin "A3"
 		)
@@
 					(unit 1)
 				)
+			)
+		)
+	)
+	(symbol
+		(lib_id "power:GND")
+		(at 40.64 35.56 90)
+		(unit 1)
+		(exclude_from_sim no)
+		(in_bom yes)
+		(on_board yes)
+		(dnp no)
+		(fields_autoplaced yes)
+		(property "Reference" "#PWR034"
+			(at 46.99 35.56 0)
+			(effects
+				(font
+					(size 1.27 1.27)
+				)
+				(hide yes)
+			)
+		)
+		(property "Value" "GND"
+			(at 43.815 35.56 90)
+			(effects
+				(font
+					(size 1.27 1.27)
+				)
+				(justify right)
+			)
+		)
+		(property "Footprint" ""
+			(at 40.64 35.56 0)
+			(effects
+				(font
+					(size 1.27 1.27)
+				)
+				(hide yes)
+			)
+		)
+		(property "Datasheet" ""
+			(at 40.64 35.56 0)
+			(effects
+				(font
+					(size 1.27 1.27)
+				)
+				(hide yes)
+			)
+		)
+		(property "Description" "Power symbol creates a global label with name \"GND\" , ground"
+			(at 40.64 35.56 0)
+			(effects
+				(font
+					(size 1.27 1.27)
+				)
+				(hide yes)
+			)
+		)
+		(pin "1"
+		)
+		(instances
+			(project "4in-2out_1.0"
+				(path "/e17a8f7c-290a-48c4-8119-0faa75a2ce74"
+					(reference "#PWR034")
+					(unit 1)
+				)

Commit message: finally standardize selected parts on all boards
Parts:
- J4: value EIB_WAGO_243-211 -> WAGO-243-211
Changed lines of the file:
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@@
 			)
 		)
-		(property "Value" "EIB_WAGO_243-211"
+		(property "Value" "WAGO-243-211"
 			(at 23.3681 109.1621 0)
 			(effects

Commit message: final for manufacturing
Parts:
- J2: footprint TerminalBlock_Phoenix:TerminalBlock_Phoenix_PT-1,5-4-3.5-H_1x04_P3.50mm_Horizontal -> TerminalBlock_Phoenix:TerminalBlock_Phoenix_PTSM-0,5-4-2.5-H-THR_1x04_P2.50mm_Horizontal
- J3: now left out of the parts list
- R1: value 680 -> 680 500mW
Changed lines of the file:
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@@
 			)
 		)
-		(property "Value" "680"
+		(property "Value" "680 500mW"
 			(at 128.27 118.8338 90)
 			(effects
@@
 			)
 		)
-		(property "Footprint" "TerminalBlock_Phoenix:TerminalBlock_Phoenix_PT-1,5-4-3.5-H_1x04_P3.50mm_Horizontal"
+		(property "Footprint" "TerminalBlock_Phoenix:TerminalBlock_Phoenix_PTSM-0,5-4-2.5-H-THR_1x04_P2.50mm_Horizontal"
 			(at 290.83 49.53 0)
 			(effects
@@
 		(unit 1)
 		(exclude_from_sim no)
-		(in_bom yes)
+		(in_bom no)
 		(on_board no)
 		(dnp yes)

Commit message: update in-out_4x-2x_2MU
Parts:
- D8: now not fitted
- R1: value 680 500mW -> 470 500mW
- SJ1, SJ2, SJ3, SJ4, SJ5, SJ6, SJ7, TP1, TP10, TP11, TP12, TP13, TP2, TP3, TP4, TP5, TP6, TP7, TP8, TP9: now left out of the parts list
Other:
- note added: "2-fach Binärausgang 230V 16A + 2- bis 4-fach Binäreingang (ARM): - Für 24V Relais R1 mit 470R bestücken, D8 nicht bestücken, SJ1 nicht brücken - Für 12V Relais R1 mit 680R bestücken, D8 nicht bestücken, SJ1 nicht brücken - Experimentell: Für 12V Relais D8 bestücken (hohe Verlustleistung an D8!) - Übliche 24V Relais: HFE20-1/24-XXXD-L2 (ggf. alternativ Omron G5RL-K1A-EL-HA DC24) (ggf. alternativ F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"
- note removed: "2-fach Binärausgang 230V 16A + 2- bis 4-fach Binäreingang (ARM): -R1 bestücken -SJ1 nicht brücken -für C1 220µF/63V verwenden -C2 nicht bestücken -24V Relais (HFE20-1/24-XXXD-L2...) verwenden (ggf. alternativ Omron G5RL-K1A-EL-HA DC24, leider single coil) (ggf. alternativ Finder 41.61.6.012.4016, bei Reichelt nur 12V und kein high inrush)"
Changed lines of the file:
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@@
 		)
 	)
-	(text "2-fach Binärausgang 230V 16A + 2- bis 4-fach Binäreingang (ARM):\n-R1 bestücken\n-SJ1 nicht brücken\n-für C1 220µF/63V verwenden\n-C2 nicht bestücken\n-24V Relais (HFE20-1/24-XXXD-L2...) verwenden\n (ggf. alternativ Omron G5RL-K1A-EL-HA DC24, leider single coil)\n (ggf. alternativ Finder 41.61.6.012.4016, bei Reichelt nur 12V und kein high inrush)"
+	(text "2-fach Binärausgang 230V 16A + 2- bis 4-fach Binäreingang (ARM):\n- Für 24V Relais R1 mit 470R bestücken, D8 nicht bestücken, SJ1 nicht brücken\n- Für 12V Relais R1 mit 680R bestücken, D8 nicht bestücken, SJ1 nicht brücken\n- Experimentell: Für 12V Relais D8 bestücken (hohe Verlustleistung an D8!)\n- Übliche 24V Relais: HFE20-1/24-XXXD-L2\n (ggf. alternativ Omron G5RL-K1A-EL-HA DC24)\n (ggf. alternativ Finder 41.61.6.012.4016)"
 		(exclude_from_sim no)
 		(at 205.74 172.72 0)
@@
 		(unit 1)
 		(exclude_from_sim no)
-		(in_bom yes)
+		(in_bom no)
 		(on_board yes)
 		(dnp no)
@@
 		(unit 1)
 		(exclude_from_sim no)
-		(in_bom yes)
+		(in_bom no)
 		(on_board yes)
 		(dnp no)
@@
 		(unit 1)
 		(exclude_from_sim no)
-		(in_bom yes)
+		(in_bom no)
 		(on_board yes)
 		(dnp no)
@@
 			)
 		)
-		(property "Value" "680 500mW"
+		(property "Value" "470 500mW"
 			(at 128.27 118.8338 90)
 			(effects
@@
 		(unit 1)
 		(exclude_from_sim no)
-		(in_bom yes)
+		(in_bom no)
 		(on_board yes)
 		(dnp no)
@@
 		(in_bom yes)
 		(on_board yes)
-		(dnp no)
+		(dnp yes)
 		(fields_autoplaced yes)
 		(property "Reference" "D8"
@@
 		(unit 1)
 		(exclude_from_sim no)
-		(in_bom yes)
+		(in_bom no)
 		(on_board yes)
 		(dnp no)
@@
 		(unit 1)
 		(exclude_from_sim no)
-		(in_bom yes)
+		(in_bom no)
 		(on_board yes)
 		(dnp no)
@@
 		(unit 1)
 		(exclude_from_sim no)
-		(in_bom yes)
+		(in_bom no)
 		(on_board yes)
 		(dnp no)
@@
 		(unit 1)
 		(exclude_from_sim no)
-		(in_bom yes)
+		(in_bom no)
 		(on_board yes)
 		(dnp no)
@@
 		(unit 1)
 		(exclude_from_sim no)
-		(in_bom yes)
+		(in_bom no)
 		(on_board yes)
 		(dnp no)
@@
 		(unit 1)
 		(exclude_from_sim no)
-		(in_bom yes)
+		(in_bom no)
 		(on_board yes)
 		(dnp no)
@@
 		(unit 1)
 		(exclude_from_sim no)
-		(in_bom yes)
+		(in_bom no)
 		(on_board yes)
 		(dnp no)
@@
 		(unit 1)
 		(exclude_from_sim no)
-		(in_bom yes)
+		(in_bom no)
 		(on_board yes)
 		(dnp no)
@@
 		(unit 1)
 		(exclude_from_sim no)
-		(in_bom yes)
+		(in_bom no)
 		(on_board yes)
 		(dnp no)
@@
 		(unit 1)
 		(exclude_from_sim no)
-		(in_bom yes)
+		(in_bom no)
 		(on_board yes)
 		(dnp no)
@@
 		(unit 1)
 		(exclude_from_sim no)
-		(in_bom yes)
+		(in_bom no)
 		(on_board yes)
 		(dnp no)
@@
 		(unit 1)
 		(exclude_from_sim no)
-		(in_bom yes)
+		(in_bom no)
 		(on_board yes)
 		(dnp no)
@@
 		(unit 1)
 		(exclude_from_sim no)
-		(in_bom yes)
+		(in_bom no)
 		(on_board yes)
 		(dnp no)
@@
 		(unit 1)
 		(exclude_from_sim no)
-		(in_bom yes)
+		(in_bom no)
 		(on_board yes)
 		(dnp no)
@@
 		(unit 1)
 		(exclude_from_sim no)
-		(in_bom yes)
+		(in_bom no)
 		(on_board yes)
 		(dnp no)
@@
 		(unit 1)
 		(exclude_from_sim no)
-		(in_bom yes)
+		(in_bom no)
 		(on_board yes)
 		(dnp no)
