File: controller_lpc1115/lpc1115_2MU_MID/lpc1115_2MU_MID_v1.04/controller_lpc1115_2MU_v1.04/controller_lpc1115_2MU_v1.04.kicad_pcb (KiCad board)
At the start: 2 copper layers, 32 x 58.1 mm, 59 parts, among them IC1 LPC1115, J1 Conn_App, J2 Conn_UI, J3 Conn_JTAG, Q1 BCP51, Q2 BC847, Q3 BC856, SW1 SW_Omron_B3FS, U1 MCP16331CH, X1 50MHz

Commit message: update controller_lpc1115_2MU_v1.04
Parts:
- added TP1: L2_IN, TestPoint:TestPoint_Pad_D1.0mm, F.Cu at (161.8, 80.0)
- added TP2: 3V3, TestPoint:TestPoint_Pad_D1.0mm, F.Cu at (156.2, 130.3)
- added TP3: EIB_DC, TestPoint:TestPoint_Pad_D1.0mm, F.Cu at (156.2, 128.0)
- added TP4: EIB_DAT, TestPoint:TestPoint_Pad_D1.0mm, F.Cu at (161.8, 83.1)
- added TP5: EIB_PU, TestPoint:TestPoint_Pad_D1.0mm, F.Cu at (154.4, 116.3)
- added TP6: EIB_OUT, TestPoint:TestPoint_Pad_D1.0mm, F.Cu at (150.1, 106.4)
- added TP7: EIB_IN, TestPoint:TestPoint_Pad_D1.0mm, F.Cu at (159.3, 78.2)
- C1, C20, C8, D1, D2, D3, Q1, R12, R16, R17, R3, R7, R8, R9: moved to F.Cu
- C10, D6, R1, R18, R2, R5: moved to B.Cu
- D5: value RB060M-60 -> RB060M-60 / MBR 140SFT1G; footprint controller_lpc1115_2MU_v1.04:SOD123 -> Diode_SMD:D_SOD-123F
- IC1: footprint controller_lpc1115_2MU_v1.04:LQFP48 -> Package_QFP:LQFP-48_7x7mm_P0.5mm
- moved D3 29.6 mm to (159.5, 89.2), turned to -90 degrees
- moved R6 20.5 mm to (153.2, 97.0), turned to 90 degrees
- moved R1 18.1 mm to (143.3, 131.3), turned to -90 degrees
- moved R14 16.0 mm to (140.0, 114.6)
- moved R2 15.2 mm to (141.0, 131.3), turned to 90 degrees
- moved R11 14.6 mm to (148.8, 94.5), turned to -90 degrees
- moved R4 11.2 mm to (151.1, 94.5), turned to -90 degrees
- moved D4 10.8 mm to (144.8, 114.6), turned to 180 degrees
- moved D10 10.3 mm to (157.0, 118.6)
- moved C9 10.0 mm to (143.8, 80.0), turned to -90 degrees
- moved D2 9.94 mm to (162.1, 89.2), turned to -90 degrees
- moved R7 9.85 mm to (156.5, 79.9), turned to 0 degrees
- moved D6 8.92 mm to (157.0, 124.2), turned to -90 degrees
- moved C8 6.97 mm to (146.1, 80.0), turned to -90 degrees
- moved R17 6.44 mm to (155.2, 97.0)
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Connections:
- C17 pad 2: Net-(U1-SW) -> Net-(D5-K)
- L1 pad 1: Net-(U1-SW) -> Net-(D5-K)
- U1 pad 6: Net-(U1-SW) -> Net-(D5-K)
Routing:
- net (no net): track 71.6 -> 0.00 mm
- net /IO12: track 2.54 -> 36.3 mm, vias 0 -> 2
- net /EIB_DC: track 34.8 -> 66.9 mm
- net /RESET: track 0.00 -> 28.8 mm, vias 1 -> 0
- net Net-(D3-K): track 0.32 -> 23.6 mm
- net Net-(Q2-B): track 32.2 -> 10.5 mm
- net /ISP_EN: track 0.00 -> 20.7 mm
- net Net-(U1-EN): track 20.2 -> 4.14 mm, vias 0 -> 1
- net Net-(Q1-C): track 0.00 -> 15.9 mm, vias 0 -> 1
- net /EIB_IN: track 32.3 -> 45.1 mm, vias 2 -> 3
- net /IO14: track 0.00 -> 12.3 mm
- net Net-(D2-A): track 17.0 -> 5.73 mm
- net Net-(D2-K): track 31.3 -> 42.5 mm, vias 3 -> 0
- net Net-(U1-SW): track 10.6 -> 0.00 mm, vias 2 -> 0
- net Net-(D5-K): track 0.00 -> 10.5 mm, vias 0 -> 1
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Other:
- board text added: "Cu"
- board text added: "LPC1115_2TE_V2.00"
- board text added: "Mask"
- board text added: "Paste"
- board text added: "Silk"
- board text removed: "+"
- board text removed: "GND"
- board text removed: "LPC1115_2TE_V1.04"
- board text removed: "Ref"
- board text removed: "TOP v1.04a CNMB"
- board text removed: "VCC"

Commit message: update
Parts:
- moved C20 44.4 mm to (178.5, 86.3), turned to 180 degrees
- moved D5 42.9 mm to (129.5, 87.9), turned to 0 degrees
- moved C17 42.8 mm to (126.1, 93.9), turned to 90 degrees
- moved R16 42.6 mm to (178.5, 88.3), turned to 0 degrees
- moved L1 42.2 mm to (130.1, 87.9), turned to 90 degrees
- moved D1 41.8 mm to (179.2, 90.6), turned to 0 degrees
- moved R10 40.5 mm to (179.7, 93.4), turned to 180 degrees
- moved R2 40.4 mm to (128.4, 92.9), turned to 0 degrees
- moved TP7 39.8 mm to (181.3, 111.4), turned to -90 degrees
- moved C9 39.2 mm to (179.7, 95.7), turned to 180 degrees
- moved R1 39.1 mm to (128.4, 95.2), turned to 180 degrees
- moved U1 39.0 mm to (128.9, 94.1), turned to 90 degrees
- moved C15 39.0 mm to (133.8, 87.0), turned to -90 degrees
- moved TP1 38.2 mm to (179.7, 113.7), turned to -90 degrees
- moved C8 38.2 mm to (179.7, 97.9), turned to 180 degrees
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Routing:
- net GND: track 16.0 -> 19.0 mm
- net Net-(Q3-B): track 8.01 -> 8.75 mm
- net +3V3: track 178.6 -> 177.9 mm
Other:
- board size 32 x 58.1 mm -> 57.5 x 32 mm
- board text added: "3V3"
- board text added: "<- upper side of rail mount enclosure HV side of application pcb"
- board text added: "EIB + input terminals ->"
- board text added: "EIB_DC"

Commit message: update controller_lpc1115_2MU_v1.04 - final for now
Parts:
- C3: footprint Capacitor_THT:CP_Radial_D5.0mm_P2.50mm -> Capacitor_SMD:CP_Elec_6.3x7.7
- C5: footprint Capacitor_THT:CP_Radial_D8.0mm_P3.50mm -> Capacitor_SMD:CP_Elec_6.3x7.7
- D4: footprint LED_THT:LED_D3.0mm -> LED_SMD:LED_1206_3216Metric
- L1: footprint Inductor_SMD:L_1812_4532Metric_Pad1.30x3.40mm_HandSolder -> Inductor_SMD:L_1812_4532Metric
- Q1: value BCP51 -> FZT753
- R14: moved to F.Cu
- SW1: footprint Button_Switch_THT:SW_TH_Tactile_Omron_B3F-10xx -> Button_Switch_SMD:SW_SPST_Omron_B3FS-100xP
- moved TP5 8.05 mm to (144.5, 114.3)
- moved C12 6.36 mm to (132.7, 99.7), turned to 180 degrees
- moved SW1 4.58 mm to (137.8, 95.1)
- moved R14 3.83 mm to (146.7, 95.4), turned to -90 degrees
- moved D4 1.49 mm to (144.3, 95.5), turned to -90 degrees
- moved R13 1.12 mm to (142.4, 89.8)
- moved C5 0.80 mm to (146.4, 104.1)
- moved C3 0.55 mm to (136.7, 87.9)
- moved L1 0.53 mm to (129.5, 87.8)
Routing:
- net /PROG: track 58.1 -> 47.5 mm, vias 2 -> 3
- net /EIB_DC: track 66.9 -> 62.8 mm, vias 2 -> 1
- net GND: track 19.0 -> 15.1 mm
- net +3V3: track 177.9 -> 181.6 mm, vias 7 -> 10
- net Net-(D10-A): track 34.3 -> 37.0 mm
- net /IO12: track 36.3 -> 37.1 mm
- net /APROG: track 23.0 -> 23.6 mm
- net Net-(D5-K): track 10.5 -> 9.94 mm
- net /IO6: track 26.4 -> 26.9 mm
- net (no net): vias 0 -> 1

Commit message: clean up controller_lpc1115_2MU_v1.04
Parts:
- added C13: 100n, Capacitor_SMD:C_0805_2012Metric, F.Cu at (128.3, 97.2)
- added D7: 1N4148W, Diode_SMD:D_SOD-123, B.Cu at (128.4, 92.8)
- added R24: 24R 1W, Resistor_SMD:R_2512_6332Metric, B.Cu at (167.6, 103.5)
- C12: value 4.7µF/50V -> 4.7µ/35V
- C15: value 10µ/10V -> 47µ/10V; footprint Capacitor_SMD:C_0805_2012Metric -> Capacitor_SMD:C_1206_3216Metric
- C16, C7: moved to B.Cu
- C17: value 15nF -> 15n
- C20: value C-EUC1206 -> 100n
- C5: value 100µ -> 100µ/35V
- D4: footprint LED_SMD:LED_1206_3216Metric -> LED_SMD:LED_0805_2012Metric
- J1: value Conn_App -> Conn_01x10; footprint Connector_PinHeader_2.54mm:PinHeader_1x09_P2.54mm_Vertical -> Connector_Molex:Molex_KK-254_AE-6410-10A_1x10_P2.54mm_Vertical; moved to B.Cu
- L1: value 6.8uH -> 10u
- L2: footprint Inductor_THT:L_Radial_D10.0mm_P5.00mm_Neosid_SD12_style3 -> selfbus:BS11_LIEGEND
- R19, R20: moved to F.Cu
- R22: value 2k4 -> 88k7; moved to B.Cu
- R23: value 680R -> 22k1; moved to B.Cu
- U1: renamed from IC1; value LPC1115 -> LPC1115FBD48-303
- U2: renamed from U1; value MCP16331CH -> TPS560430
- X1: value 50MHz -> 12MHz
- moved C7 20.5 mm to (136.4, 86.9), turned to 90 degrees
- moved R18 6.57 mm to (171.6, 106.9), turned to 0 degrees
- moved C15 4.94 mm to (138.7, 87.4), turned to 90 degrees
- moved C12 4.46 mm to (128.3, 99.3), turned to 0 degrees
- moved C17 4.22 mm to (126.1, 89.7)
- moved R20 3.02 mm to (128.3, 101.5)
- moved TP2 2.95 mm to (126.5, 108.1)
- moved R19 2.64 mm to (128.3, 103.6), turned to 0 degrees
- moved J1 2.55 mm to (168.3, 111.8), turned to 180 degrees
- moved L2 2.48 mm to (138.2, 114.3)
- moved C16 2.46 mm to (128.3, 103.1)
- moved R2 2.14 mm to (128.3, 95.0), turned to 180 degrees
- moved R22 2.12 mm to (128.3, 101.1)
- moved D6 1.92 mm to (135.1, 110.7)
- moved D10 1.92 mm to (140.7, 110.7)
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Connections:
- J1 pad 1: Net-(D2-A) -> GND
- J1 pad 2: GND -> Net-(D2-A)
- J1 pad 3: +3V3 -> GND
- J1 pad 4: /PWM -> +3V3
- J1 pad 5: /IO7 -> /PWM
- J1 pad 6: /IO5 -> /IO7
- J1 pad 7: /IO6 -> /IO5
- J1 pad 8: /APROG -> /IO6
- J1 pad 9: /EIB_DC -> /APROG
- Q2 pad 2: Net-(Q1-C) -> Net-(Q2-E)
- R18 pad 1: Net-(Q1-C) -> Net-(Q2-E)
Routing:
- net Net-(Q1-C): track 15.9 -> 4.12 mm
- net Net-(Q2-E): track 0.00 -> 4.98 mm, vias 0 -> 1
- net +3V3: track 181.6 -> 186.4 mm, vias 10 -> 9
- net Net-(D2-A): track 5.73 -> 9.14 mm
- net Net-(U2-V_{FB}): track 12.4 -> 9.10 mm, vias 0 -> 1
- net Net-(D7-K): track 2.03 -> 4.15 mm, vias 0 -> 1
- net Net-(Q2-B): track 10.5 -> 12.0 mm
- net /EIB_DC: track 62.8 -> 64.3 mm
- net Net-(D5-K): track 9.94 -> 11.2 mm
- net /PROG: track 47.5 -> 48.5 mm
- net Net-(C4-Pad2): track 4.19 -> 3.30 mm
- net /IO12: track 37.1 -> 37.8 mm, vias 2 -> 3
- net /APROG: track 23.6 -> 24.2 mm
- net /IO6: track 26.9 -> 27.5 mm
- net (no net): vias 1 -> 0
- added copper zone on F.Cu, net Net-(Q1-C)
