File: controller_lpc1115/lpc1115_2MU_MID/lpc1115_2MU_MID_v1.04/controller_lpc1115_2MU_v1.04/controller_lpc1115_2MU_v1.04.kicad_sch (KiCad schematic)
At the start: 59 parts, among them IC1 LPC1115, J1 Conn_App, J2 Conn_UI, J3 Conn_JTAG, Q1 BCP51, Q2 BC847, Q3 BC856, SW1 SW_Omron_B3FS, U1 MCP16331CH, X1 50MHz

Commit message: update controller_lpc1115_2MU_v1.04
Parts:
- added TP1: L2_IN, TestPoint:TestPoint_Pad_D1.0mm, symbol Connector:TestPoint
- added TP2: 3V3, TestPoint:TestPoint_Pad_D1.0mm, symbol Connector:TestPoint
- added TP3: EIB_DC, TestPoint:TestPoint_Pad_D1.0mm, symbol Connector:TestPoint
- added TP4: EIB_DAT, TestPoint:TestPoint_Pad_D1.0mm, symbol Connector:TestPoint
- added TP5: EIB_PU, TestPoint:TestPoint_Pad_D1.0mm, symbol Connector:TestPoint
- added TP6: EIB_OUT, TestPoint:TestPoint_Pad_D1.0mm, symbol Connector:TestPoint
- added TP7: EIB_IN, TestPoint:TestPoint_Pad_D1.0mm, symbol Connector:TestPoint
Connections:
- net +3V3: now also TP2.1
- net EIB_DC: now also TP3.1
- net EIB_IN: now also TP7.1
- net EIB_OUT: now also TP6.1
- net at C10.2, D3.1 (K), Q1.3 (E)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: now also TP4.1
- net at D10.2 (A), R11.2, R4.2: now also TP5.1
- net at D2.1 (K), L2.1: now also TP1.1
Other:
- moved on the sheet: D10

Commit message: update controller_lpc1115_2MU_v1.04 - final for now
Parts:
- C3: footprint Capacitor_THT:CP_Radial_D5.0mm_P2.50mm -> Capacitor_SMD:CP_Elec_6.3x7.7
- C5: footprint Capacitor_THT:CP_Radial_D8.0mm_P3.50mm -> Capacitor_SMD:CP_Elec_6.3x7.7
- D4: footprint LED_THT:LED_D3.0mm -> LED_SMD:LED_1206_3216Metric
- L1: footprint Inductor_SMD:L_1812_4532Metric_Pad1.30x3.40mm_HandSolder -> Inductor_SMD:L_1812_4532Metric
- Q1: value BCP51 -> FZT753; symbol Transistor_BJT:BCP51 -> Device:Q_PNP_BCE
- SW1: footprint Button_Switch_THT:SW_TH_Tactile_Omron_B3F-10xx -> Button_Switch_SMD:SW_SPST_Omron_B3FS-100xP
Changed lines of the file:
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@@
 	)
 	(symbol
-		(lib_id "Transistor_BJT:BCP51")
+		(lib_id "Device:Q_PNP_BCE")
 		(at 71.12 182.88 180)
 		(unit 1)
@@
 			)
 		)
-		(property "Value" "BCP51"
+		(property "Value" "FZT753"
 			(at 66.2686 184.4422 0)
 			(effects
@@
 		)
 		(property "Footprint" "Package_TO_SOT_SMD:SOT-223-3_TabPin2"
-			(at 66.04 180.975 0)
+			(at 66.04 185.42 0)
 			(effects
 				(font
 					(size 1.27 1.27)
-					(italic yes)
 				)
-				(justify left)
 				(hide yes)
 			)
 		)
-		(property "Datasheet" "https://www.onsemi.com/pub/Collateral/BCP51-D.pdf"
+		(property "Datasheet" "~"
 			(at 71.12 182.88 0)
 			(effects
@@
 					(size 1.27 1.27)
 				)
-				(justify left)
 				(hide yes)
 			)
 		)
-		(property "Description" ""
+		(property "Description" "PNP transistor, base/collector/emitter"
 			(at 71.12 182.88 0)
 			(effects
@@
 			)
 		)
-		(property "Footprint" "Capacitor_THT:CP_Radial_D8.0mm_P3.50mm"
+		(property "Footprint" "Capacitor_SMD:CP_Elec_6.3x7.7"
 			(at 102.5652 149.86 0)
 			(effects
@@
 		(on_board yes)
 		(dnp no)
+		(fields_autoplaced yes)
 		(property "Reference" "R22"
-			(at 107.95 57.0106 90)
+			(at 107.95 53.8862 90)
 			(effects
 				(font
@@
 		)
 		(property "Value" "2k4"
-			(at 107.95 53.8862 90)
+			(at 107.95 57.0106 90)
 			(effects
 				(font
@@
 			)
 		)
-		(property "Footprint" "Capacitor_THT:CP_Radial_D5.0mm_P2.50mm"
+		(property "Footprint" "Capacitor_SMD:CP_Elec_6.3x7.7"
 			(at 168.6052 81.28 0)
 			(effects
@@
 			)
 		)
-		(property "Footprint" "Button_Switch_THT:SW_TH_Tactile_Omron_B3F-10xx"
+		(property "Footprint" "Button_Switch_SMD:SW_SPST_Omron_B3FS-100xP"
 			(at 104.14 228.6 0)
 			(effects
@@
 			)
 		)
-		(property "Footprint" "LED_THT:LED_D3.0mm"
+		(property "Footprint" "LED_SMD:LED_1206_3216Metric"
 			(at 86.36 233.68 0)
 			(effects
@@
 			)
 		)
-		(property "Footprint" "Inductor_SMD:L_1812_4532Metric_Pad1.30x3.40mm_HandSolder"
+		(property "Footprint" "Inductor_SMD:L_1812_4532Metric"
 			(at 115.57 63.5 0)
 			(effects

Commit message: clean up controller_lpc1115_2MU_v1.04
Parts:
- added C13: 100n, Capacitor_SMD:C_0805_2012Metric, symbol Device:C
- added D7: 1N4148W, Diode_SMD:D_SOD-123, symbol Diode:1N4148W
- added R24: 24R 1W, Resistor_SMD:R_2512_6332Metric, symbol Device:R
- C12: value 4.7µF/50V -> 4.7µ/35V
- C15: value 10µ/10V -> 47µ/10V; footprint Capacitor_SMD:C_0805_2012Metric -> Capacitor_SMD:C_1206_3216Metric
- C16: now not fitted
- C17: value 15nF -> 15n
- C20: value C-EUC1206 -> 100n
- C5: value 100µ -> 100µ/35V
- D4: footprint LED_SMD:LED_1206_3216Metric -> LED_SMD:LED_0805_2012Metric
- J1: value Conn_App -> Conn_01x10; footprint Connector_PinHeader_2.54mm:PinHeader_1x09_P2.54mm_Vertical -> Connector_Molex:Molex_KK-254_AE-6410-10A_1x10_P2.54mm_Vertical; symbol Connector_Generic:Conn_01x09 -> Connector_Generic:Conn_01x10
- L1: value 6.8uH -> 10u
- L2: footprint Inductor_THT:L_Radial_D10.0mm_P5.00mm_Neosid_SD12_style3 -> selfbus:BS11_LIEGEND
- R22: value 2k4 -> 88k7
- R23: value 680R -> 22k1
- U1: renamed from IC1; value LPC1115 -> LPC1115FBD48-303
- U2: renamed from U1; value MCP16331CH -> TPS560430; symbol Regulator_Switching:MCP16331CH -> Regulator_Switching:MCP16331x-xCH
- X1: value 50MHz -> 12MHz
Connections:
- net +3V3: now also J1.4 (Pin_4), D7.2 (A); no longer J1.3 (Pin_3)
- net APROG: now also J1.9 (Pin_9); no longer J1.8 (Pin_8)
- net EIB_DC: now also J1.10 (Pin_10), C13.2; no longer J1.9 (Pin_9)
- net GND: now also J1.1 (Pin_1), J1.3 (Pin_3), C13.1; no longer J1.2 (Pin_2)
- net IO5: now also J1.7 (Pin_7); no longer J1.6 (Pin_6)
- net IO6: now also J1.8 (Pin_8); no longer J1.7 (Pin_7)
- net IO7: now also J1.6 (Pin_6); no longer J1.5 (Pin_5)
- net PWM: now also J1.5 (Pin_5); no longer J1.4 (Pin_4)
- net at Q2.2 (E), R18.1: now also R24.2; no longer Q1.2 (C)
- net at C17.1, U2.1 (BOOST): now also D7.1 (K)
- net at D2.2 (A), D3.2 (A): now also J1.2 (Pin_2); no longer J1.1 (Pin_1)
- new net: Q1.2 (C), R24.1
Other:
- note added: "Power LED (D4+R14) ist optional"
- note added: "für Rohm BD9G101: R22=4k4, R23=680, C16=270n, D7 nicht bestücken für MCP16331: R22=31,25k, R23=10k, C16 nicht bestücken, D7 bestücken für TPS560430: R22=88,7k, R23=22,1k, C16 nicht bestücken, D7 nicht bestücken"
- note removed: "Power LED (LED4+R20) ist optional"
- moved on the sheet: C12, C15, C17, C20, C3, C5, C6, C7, D1, D5, L1, R16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
