File: controller_lpc1115/lpc1115_2MU_MID/lpc1115_2MU_MID_kicad/controller_lpc1115_2MU_v1.04.kicad_sch (KiCad schematic)
At the start: 69 parts, among them J1 Conn_01x10, J2 Conn_UI, J3 Conn_JTAG, Q1 FZT753, Q2 BC847, Q3 BC856, SW1 SW_Omron_B3FS, U1 LPC1115FBD48-303, U2 TPS560430, X1 12MHz

Commit message: fixups for 2MU/4MU controllers - use Seiko oszillator
Parts:
- J3: footprint Connector_PinSocket_2.00mm:PinSocket_2x05_P2.00mm_Vertical -> Connector_PinHeader_2.00mm:PinHeader_2x05_P2.00mm_Vertical
- X1: footprint Oscillator:Oscillator_SMD_EuroQuartz_XO32-4Pin_3.2x2.5mm -> Oscillator:Oscillator_SMD_SeikoEpson_SG210-4Pin_2.5x2.0mm; symbol Oscillator:XO32 -> Oscillator:SG-210STF
Changed lines of the file:
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@@
 		)
 		(instances
-			(project ""
+			(project "controller_lpc1115_2MU_v1.04"
 				(path "/60be9403-0258-4972-a31b-1601aa9cd87c"
 					(reference "R24")
@@
 			)
 		)
-		(property "Footprint" "Connector_PinSocket_2.00mm:PinSocket_2x05_P2.00mm_Vertical"
+		(property "Footprint" "Connector_PinHeader_2.00mm:PinHeader_2x05_P2.00mm_Vertical"
 			(at 317.5 68.58 0)
 			(effects
@@
 	)
 	(symbol
-		(lib_id "Oscillator:XO32")
+		(lib_id "Oscillator:SG-210STF")
 		(at 223.52 172.72 0)
 		(unit 1)
@@
 		(fields_autoplaced yes)
 		(property "Reference" "X1"
-			(at 232.5877 166.575 0)
+			(at 233.68 166.4014 0)
 			(effects
 				(font
@@
 		)
 		(property "Value" "12MHz"
-			(at 232.5877 168.9993 0)
+			(at 233.68 168.9414 0)
 			(effects
 				(font
@@
 			)
 		)
-		(property "Footprint" "Oscillator:Oscillator_SMD_EuroQuartz_XO32-4Pin_3.2x2.5mm"
-			(at 241.3 181.61 0)
+		(property "Footprint" "Oscillator:Oscillator_SMD_SeikoEpson_SG210-4Pin_2.5x2.0mm"
+			(at 234.95 181.61 0)
 			(effects
 				(font
@@
 			)
 		)
-		(property "Datasheet" "http://cdn-reichelt.de/documents/datenblatt/B400/XO32.pdf"
+		(property "Datasheet" "https://support.epson.biz/td/api/doc_check.php?mode=dl&lang=en&Parts=SG-210STF"
 			(at 220.98 172.72 0)
 			(effects
@@
 			)
 		)
-		(property "Description" "HCMOS Clock Oscillator"
+		(property "Description" "CMOS Crystal Oscillator SPXO"
 			(at 223.52 172.72 0)
 			(effects
@@
 		)
 		(instances
-			(project ""
+			(project "controller_lpc1115_2MU_v1.04"
 				(path "/60be9403-0258-4972-a31b-1601aa9cd87c"
 					(reference "D7")

Commit message: finally standardize selected parts on all boards
Parts:
- C12: value 4.7µ/35V -> 4.7u/35V
- C15: value 47µ/10V -> 47u/10V
- C16, D7: now left out of the parts list
- C3: value 100µ/10V -> 100u/10V
- C5: value 100µ/35V -> 100u/35V
- D10: value 7,5V -> 7V5
- D5: footprint Diode_SMD:D_SOD-123F -> Diode_SMD:D_SOD-123
Changed lines of the file:
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@@
 		(unit 1)
 		(exclude_from_sim no)
-		(in_bom yes)
+		(in_bom no)
 		(on_board yes)
 		(dnp yes)
@@
 			)
 		)
-		(property "Value" "47µ/10V"
+		(property "Value" "47u/10V"
 			(at 133.731 75.2222 0)
 			(effects
@@
 			)
 		)
-		(property "Value" "100µ/35V"
+		(property "Value" "100u/35V"
 			(at 101.981 146.7232 0)
 			(effects
@@
 			)
 		)
-		(property "Value" "4.7µ/35V"
+		(property "Value" "4.7u/35V"
 			(at 40.259 75.2222 0)
 			(effects
@@
 			)
 		)
-		(property "Value" "100µ/10V"
+		(property "Value" "100u/10V"
 			(at 164.211 74.3332 0)
 			(effects
@@
 			)
 		)
-		(property "Value" "7,5V"
+		(property "Value" "7V5"
 			(at 86.868 166.6622 90)
 			(effects
@@
 		(unit 1)
 		(exclude_from_sim no)
-		(in_bom yes)
+		(in_bom no)
 		(on_board yes)
 		(dnp yes)
@@
 			)
 		)
-		(property "Footprint" "Diode_SMD:D_SOD-123F"
+		(property "Footprint" "Diode_SMD:D_SOD-123"
 			(at 102.87 76.2 0)
 			(effects

Commit message: final for manufacturing
Parts:
- R13: value 91k -> 43k
- R16: value 10k -> 6k2
- R22: value 88k7 -> 51k
Connections:
- net EIB_DC: now also D10.1 (K); no longer D6.2 (A), R13.1
- net at R11.2, R4.2, TP5.1: now also D6.1 (K); no longer D10.2 (A)
- new net: D10.2 (A), D6.2 (A), R13.1
Other:
- note added: "für Rohm BD9G101: R22=4k4, R23=680, C16=270n, D7 nicht bestücken für MCP16331: R22=31,25k, R23=10k, C16 nicht bestücken, D7 bestücken für TPS560430: R22=51k, R23=22,1k, C16 nicht bestücken, D7 nicht bestücken"
- note removed: "für Rohm BD9G101: R22=4k4, R23=680, C16=270n, D7 nicht bestücken für MCP16331: R22=31,25k, R23=10k, C16 nicht bestücken, D7 bestücken für TPS560430: R22=88,7k, R23=22,1k, C16 nicht bestücken, D7 nicht bestücken"
- moved on the sheet: C20, C5, D1, D10, D6, R13, R16

Commit message: update controller_lpc1115_2MU_v1.04
Parts:
- C17: value 15n -> 100n
- TP1, TP2, TP3, TP4, TP5, TP6, TP7: now left out of the parts list
Changed lines of the file:
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@@
 		(unit 1)
 		(exclude_from_sim no)
-		(in_bom yes)
+		(in_bom no)
 		(on_board yes)
 		(dnp no)
@@
 			)
 		)
-		(property "Value" "15n"
+		(property "Value" "100n"
 			(at 96.52 56.7308 90)
 			(effects
@@
 		(unit 1)
 		(exclude_from_sim no)
-		(in_bom yes)
+		(in_bom no)
 		(on_board yes)
 		(dnp no)
@@
 		(unit 1)
 		(exclude_from_sim no)
-		(in_bom yes)
+		(in_bom no)
 		(on_board yes)
 		(dnp no)
@@
 		(unit 1)
 		(exclude_from_sim no)
-		(in_bom yes)
+		(in_bom no)
 		(on_board yes)
 		(dnp no)
@@
 		(unit 1)
 		(exclude_from_sim no)
-		(in_bom yes)
+		(in_bom no)
 		(on_board yes)
 		(dnp no)
@@
 		(unit 1)
 		(exclude_from_sim no)
-		(in_bom yes)
+		(in_bom no)
 		(on_board yes)
 		(dnp no)
@@
 		(unit 1)
 		(exclude_from_sim no)
-		(in_bom yes)
+		(in_bom no)
 		(on_board yes)
 		(dnp no)

Commit message: update xtal caps, eib_in cap+resistor, bus_v resistors
Parts:
- C18: value 100p -> 22p
- C2: value 220p -> 22p
- R13, R16: now not fitted; now left out of the parts list
- R8: value 47k -> 100k
Changed lines of the file:
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@@
 	)
 	(junction
-		(at 81.28 86.36)
-		(diameter 0)
-		(color 0 0 0 0)
-	)
-	(junction
 		(at 139.7 60.96)
 		(diameter 0)
@@
 	(wire
 		(pts
-			(xy 81.28 86.36) (xy 81.28 87.63)
+			(xy 80.01 86.36) (xy 80.01 87.63)
 		)
 		(stroke
@@
 	(wire
 		(pts
-			(xy 80.01 86.36) (xy 81.28 86.36)
+			(xy 80.01 86.36) (xy 102.87 86.36)
 		)
 		(stroke
@@
 	(wire
 		(pts
-			(xy 81.28 86.36) (xy 102.87 86.36)
-		)
-		(stroke
-			(width 0.1524)
-			(type solid)
-		)
-	)
-	(wire
-		(pts
 			(xy 68.58 170.18) (xy 78.74 170.18)
 		)
@@
 		(unit 1)
 		(exclude_from_sim no)
-		(in_bom yes)
+		(in_bom no)
 		(on_board yes)
-		(dnp no)
+		(dnp yes)
 		(fields_autoplaced yes)
 		(property "Reference" "R13"
@@
 			)
 		)
-		(property "Value" "47k"
+		(property "Value" "100k"
 			(at 133.858 166.6622 0)
 			(effects
@@
 		(unit 1)
 		(exclude_from_sim no)
-		(in_bom yes)
+		(in_bom no)
 		(on_board yes)
-		(dnp no)
+		(dnp yes)
 		(fields_autoplaced yes)
 		(property "Reference" "R16"
@@
 	(symbol
 		(lib_id "power:GND")
-		(at 81.28 87.63 0)
+		(at 80.01 87.63 0)
 		(unit 1)
 		(exclude_from_sim no)
@@
 		(fields_autoplaced yes)
 		(property "Reference" "#GND03"
-			(at 81.28 87.63 0)
+			(at 80.01 87.63 0)
 			(effects
 				(font
@@
 		)
 		(property "Value" "GND"
-			(at 81.28 92.1132 0)
+			(at 80.01 92.1132 0)
 			(effects
 				(font
@@
 		)
 		(property "Footprint" ""
-			(at 81.28 87.63 0)
+			(at 80.01 87.63 0)
 			(effects
 				(font
@@
 		)
 		(property "Datasheet" ""
-			(at 81.28 87.63 0)
+			(at 80.01 87.63 0)
 			(effects
 				(font
@@
 		)
 		(property "Description" ""
-			(at 81.28 87.63 0)
+			(at 80.01 87.63 0)
 			(effects
 				(font
@@
 		(fields_autoplaced yes)
 		(property "Reference" "C18"
-			(at 243.459 164.8078 0)
+			(at 249.301 164.8078 0)
 			(effects
 				(font
 					(size 1.778 1.5113)
 				)
-				(justify left)
+				(justify right)
 			)
 		)
-		(property "Value" "100p"
-			(at 243.459 167.9322 0)
+		(property "Value" "22p"
+			(at 249.301 167.9322 0)
 			(effects
 				(font
 					(size 1.778 1.5113)
 				)
-				(justify left)
+				(justify right)
 			)
 		)
@@
 			)
 		)
-		(property "Value" "220p"
+		(property "Value" "22p"
 			(at 259.461 167.9322 0)
 			(effects
