File: controller_lpc1115/lpc1115_2MU_MID/lpc1115_2MU_MID_kicad/lpc1115_2MU_MID.kicad_pcb (KiCad board)
At the start: 2 copper layers, 57.5 x 32 mm, 69 parts, among them J1 Conn_01x10, J2 Conn_UI, J3 Conn_JTAG, Q1 FZT753, Q2 BC847, Q3 BC856, SW1 SW_Omron_B3FS, U1 LPC1115FBD48-303, U2 TPS560430, X1 12MHz

Commit message: rename controller_lpc1115_2MU_v1.04 -> lpc1115_2MU_MID
version 2.01
Other:
- board text added: "LPC1115_2TE_V2.01"
- board text removed: "LPC1115_2TE_V2.00"
