File: controller_lpc1115/lpc1115_2MU_MID/lpc1115_2MU_MID_kicad/lpc1115_2MU_MID.kicad_sch (KiCad schematic)
At the start: 69 parts, among them J1 Conn_01x10, J2 Conn_UI, J3 Conn_JTAG, Q1 FZT753, Q2 BC847, Q3 BC856, SW1 SW_Omron_B3FS, U1 LPC1115FBD48-303, U2 TPS560430, X1 12MHz

Commit message: controllers: reduce osc load, fix DNP for voltage measurement
Parts:
- R13, R16: now fitted; now in the parts list
Changed lines of the file:
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@@
 		(unit 1)
 		(exclude_from_sim no)
-		(in_bom no)
-		(on_board yes)
-		(dnp yes)
+		(in_bom yes)
+		(on_board yes)
+		(dnp no)
 		(fields_autoplaced yes)
 		(property "Reference" "R13"
@@
 		(unit 1)
 		(exclude_from_sim no)
-		(in_bom no)
-		(on_board yes)
-		(dnp yes)
+		(in_bom yes)
+		(on_board yes)
+		(dnp no)
 		(fields_autoplaced yes)
 		(property "Reference" "R16"
