File: breakout-boards/pwr_knx_v-measure/bb_pwr_knx_v-measure/bb_pwr_knx_v-measure.kicad_pcb (KiCad board)
At the start: 2 copper layers, 28.5 x 25 mm, 47 parts, among them IC100 BD9G101, T1 BC856, T2 BCP52, T3 BC847

Commit message: bump bb_pwr_knx_v WIP
Parts:
- removed JP3: , bb_pwr_knx_v-measure:1X02
- added C7: 100n, Capacitor_SMD:C_0805_2012Metric, F.Cu at (126.2, 104.8)
- added D8: 1N4148W, Diode_SMD:D_SOD-123, F.Cu at (159.3, 114.8)
- added R14: 390k, Resistor_SMD:R_0805_2012Metric, F.Cu at (121.7, 101.4)
- added R15: 43k, Resistor_SMD:R_0805_2012Metric, F.Cu at (121.7, 104.3)
- C1: value 100uF 35V -> 100µ/35V; footprint bb_pwr_knx_v-measure:SANYO-OSCON_SMD_C6_334 -> Capacitor_SMD:CP_Elec_6.3x7.7
- C10, C104, C2, C6: value 100nF -> 100n; footprint bb_pwr_knx_v-measure:C0805_334 -> Capacitor_SMD:C_0805_2012Metric
- C100: value 4.7uF 50V -> 4.7µ/35V; footprint bb_pwr_knx_v-measure:C0805_334 -> Capacitor_SMD:C_0805_2012Metric
- C101: value 470nF -> 270n; footprint bb_pwr_knx_v-measure:C0805_334 -> Capacitor_SMD:C_0805_2012Metric
- C102: value 15nF -> 15n; footprint bb_pwr_knx_v-measure:C0805_334 -> Capacitor_SMD:C_0805_2012Metric
- C103, C105: value 47uF 10V -> 47µ/10V; footprint bb_pwr_knx_v-measure:C0805_334 -> Capacitor_SMD:C_1206_3216Metric
- C3, C4: value 10nF -> 10n; footprint bb_pwr_knx_v-measure:C0805_334 -> Capacitor_SMD:C_0805_2012Metric
- C5: value 100pF -> 100p; footprint bb_pwr_knx_v-measure:C0805_334 -> Capacitor_SMD:C_0805_2012Metric
- D1: footprint bb_pwr_knx_v-measure:DO214AC -> Diode_SMD:D_SMA
- D100: value MBRS1100 -> RB060M-60 / MBR 140SFT1G; footprint bb_pwr_knx_v-measure:SOD-123 -> Diode_SMD:D_SOD-123
- D2, D3, D5: value 1N4148 -> 1N4148W; footprint bb_pwr_knx_v-measure:SOD-123 -> Diode_SMD:D_SOD-123
- D4: value 1N4148 -> 1N4148W; footprint bb_pwr_knx_v-measure:SOD-123 -> Diode_SMD:D_SOD-123; moved to B.Cu
- D6: footprint bb_pwr_knx_v-measure:SOD-123 -> Diode_SMD:D_SOD-123
- D7: value DDZ9685 -> 3V6; footprint bb_pwr_knx_v-measure:SOD-123 -> Diode_SMD:D_SOD-123
- IC100: value BD9G101 -> TPS560430; footprint bb_pwr_knx_v-measure:SOT23-6 -> Package_TO_SOT_SMD:SOT-23-6
- JP2: value (none) -> Conn_01x03_Pin; footprint bb_pwr_knx_v-measure:1X03 -> Connector_PinHeader_2.54mm:PinHeader_1x05_P2.54mm_Vertical
- JP4: value (none) -> Conn_01x02_Pin; footprint bb_pwr_knx_v-measure:1X02 -> Connector_PinHeader_2.54mm:PinHeader_1x02_P2.54mm_Vertical
- KNX0: footprint bb_pwr_knx_v-measure:WAGO-243-211 -> selfbus:W243-211_1x02_P5.75
- L1: footprint bb_pwr_knx_v-measure:BS11 -> selfbus:BS11_LIEGEND
- L100: value 4.7uH -> 10u; footprint bb_pwr_knx_v-measure:L4532P -> Inductor_SMD:L_1812_4532Metric
- R1, R10, R11, R12, R13, R2, R3, R4, R5, R6, R7, R8, R9: footprint bb_pwr_knx_v-measure:R0805_334 -> Resistor_SMD:R_0805_2012Metric
- R101: value 1k6 -> 88k7; footprint bb_pwr_knx_v-measure:R0805_334 -> Resistor_SMD:R_0805_2012Metric
- R102: value 470R -> 22k1; footprint bb_pwr_knx_v-measure:R0805_334 -> Resistor_SMD:R_0805_2012Metric
- R25: value 24R 2512 1.0W -> 24R 1W; footprint bb_pwr_knx_v-measure:R2512_334 -> Resistor_SMD:R_1206_3216Metric
- T1: footprint bb_pwr_knx_v-measure:SOT23-BEC_399 -> Package_TO_SOT_SMD:SOT-23
- T2: value BCP52 -> FZT753; footprint bb_pwr_knx_v-measure:SOT223_399 -> Package_TO_SOT_SMD:SOT-223-3_TabPin2
- T3: footprint bb_pwr_knx_v-measure:SOT23_402 -> Package_TO_SOT_SMD:SOT-23
- moved D4 10.6 mm to (141.4, 98.7)
- moved JP2 7.62 mm to (150.4, 116.2), turned to -90 degrees
- moved KNX0 5.31 mm to (155.7, 101.9), turned to 90 degrees
- moved L100 3.15 mm to (154.7, 114.4), turned to -90 degrees
- moved D100 3.06 mm to (155.3, 109.1), turned to 90 degrees
- moved C100 2.67 mm to (153.2, 108.5)
- moved D1 1.74 mm to (157.4, 98.9), turned to 180 degrees
- moved C102 1.37 mm to (158.6, 112.5)
- moved JP4 1.25 mm to (143.3, 93.8), turned to 90 degrees
- moved T2 1.20 mm to (148.5, 99.6), turned to 180 degrees
- moved R101 1.13 mm to (158.8, 106.9), turned to 180 degrees
- moved C101 0.70 mm to (161.6, 105.5)
- moved C104 0.48 mm to (149.4, 108.5)
- turned C1 to -90 degrees
- turned IC100 to 180 degrees
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Connections:
- net BST renamed Net-(D8-K)
- net FB renamed Net-(IC100-V_{FB})
- C10 pad 2: BUS_V -> /BUS_V
- C100 pad 2: EIB_DC -> /EIB_DC
- C102 pad 1: LX -> Net-(D100-K)
- C2 pad 1: N$14 -> Net-(T1-B)
- C2 pad 2: N$1 -> Net-(C2-Pad2)
- C3 pad 1: EIB+DIR -> /EIB+DIR
- C4 pad 2: EIB_OUT -> /EIB_OUT
- C5 pad 2: EIB_IN -> /EIB_IN
- C6 pad 1: GND -> /EIB_IN
- IC100 pad 4: EIB_DC -> Net-(IC100-EN)
- IC100 pad 5: EIB_DC -> /EIB_DC
- IC100 pad 6: LX -> Net-(D100-K)
- JP2 pad 1: EIB_OUT -> GND
- JP2 pad 2: BUS_V -> +3V3
- JP2 pad 3: EIB_IN -> /EIB_IN
- JP4 pad 1: N$8 -> /N$8
- JP4 pad 2: N$8 -> /N$8
- L1 pad 1: EIB_DC -> /EIB_DC
- L1 pad 2: N$2 -> Net-(D3-K)
- L100 pad 1: LX -> Net-(D100-K)
- R1 pad 1: EIB+DIR -> /EIB+DIR
- R10 pad 1: N$1 -> Net-(C2-Pad2)
- R10 pad 2: EIB+DIR -> /EIB+DIR
- R11 pad 2: EIB+DIR -> /EIB+DIR
- R12 pad 1: REF -> /REF
- R12 pad 2: BUS_V -> /BUS_V
- R13 pad 1: BUS_V -> /BUS_V
- R25 pad 2: N$8 -> /N$8
- R3 pad 1: N$25 -> Net-(D5-K)
- R4 pad 2: N$25 -> Net-(D5-K)
- R7 pad 1: EIB_IN -> /EIB_IN
- R8 pad 1: N$14 -> Net-(T1-B)
- R9 pad 2: N$14 -> Net-(T1-B)
- T2 pad 2: N$8 -> /N$8
- T2 pad 3: EIB+DIR -> /EIB+DIR
Routing:
- net EIB_DC: track 33.6 -> 0.00 mm
- net /EIB+: track 0.00 -> 31.5 mm, vias 0 -> 1
- net /EIB_DC: track 0.00 -> 31.2 mm
- net EIB+: track 21.7 -> 0.00 mm
- net /EIB+DIR: track 0.00 -> 16.0 mm, vias 0 -> 1
- net Net-(T1-B): track 0.00 -> 16.0 mm, vias 0 -> 1
- net N$14: track 15.9 -> 0.00 mm
- net EIB+DIR: track 15.1 -> 0.00 mm, vias 1 -> 0
- net Net-(T2-B): track 13.7 -> 0.00 mm
- net BUS_V: track 13.3 -> 0.00 mm
- net /BUS_V: track 0.00 -> 13.2 mm
- net N$1: track 13.0 -> 0.00 mm, vias 1 -> 0
- net Net-(D3-K): track 0.00 -> 9.28 mm
- net EIB_IN: track 8.77 -> 0.00 mm
- net GND: track 11.9 -> 3.26 mm, vias 17 -> 14
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- added copper zone on B.Cu, net /N$8
- added copper zone on F.Cu, net /N$8
- added copper zone on F.Cu, net Net-(D100-K)
- removed copper zone on F.Cu, net EIB_DC
- removed copper zone on F.Cu, net LX
- removed copper zone on B.Cu, net N$8
- removed copper zone on F.Cu, net N$8
- removed copper zone on F.Cu, net Net-(D8-K)

Commit message: bb_pwr_knx_v-measure final
Parts:
- C11: renamed from C101; moved to B.Cu
- C8: renamed from C7; moved to B.Cu
- R14, R15: moved to B.Cu
- moved R14 33.2 mm to (153.9, 109.7), turned to -90 degrees
- moved C8 31.1 mm to (156.7, 110.5)
- moved R15 30.6 mm to (151.9, 109.7), turned to 90 degrees
- moved C3 5.93 mm to (146.8, 101.9), turned to 180 degrees
- moved R1 3.80 mm to (146.8, 103.9), turned to 180 degrees
- moved R11 3.68 mm to (159.0, 102.6), turned to 90 degrees
- moved C6 3.43 mm to (144.8, 111.4)
- moved C11 2.69 mm to (159.0, 106.2)
- moved T1 2.35 mm to (144.8, 108.5), turned to 90 degrees
- moved R3 2.24 mm to (144.3, 99.1), turned to 0 degrees
- moved C2 1.46 mm to (161.0, 106.2), turned to 90 degrees
- moved R10 1.46 mm to (161.0, 102.6), turned to 90 degrees
- moved D3 1.34 mm to (140.1, 98.3)
- moved D4 1.34 mm to (140.1, 98.3)
- moved T2 1.28 mm to (149.5, 100.3), turned to -90 degrees
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- renumbered C104 to C12, C103 to C13, C105 to C14, C100 to C7, C102 to C9, D100 to D9, IC100 to IC1, L100 to L2, R101 to R16, R102 to R17
Connections:
- net /N$8 renamed /HEAT
Routing:
- net /EIB+: track 31.5 -> 18.6 mm, vias 1 -> 0
- net Net-(T2-B): track 0.00 -> 8.88 mm
- net Net-(IC1-EN): track 0.00 -> 5.94 mm, vias 0 -> 1
- net /EIB+DIR: track 16.0 -> 21.3 mm
- net Net-(D3-K): track 9.28 -> 5.16 mm
- net /EIB_IN: track 8.59 -> 11.7 mm
- net Net-(T1-B): track 16.0 -> 18.9 mm, vias 1 -> 0
- net Net-(T3-C): track 7.35 -> 4.55 mm
- net /EIB_DC: track 31.2 -> 33.4 mm, vias 0 -> 1
- net Net-(IC1-V_{FB}): track 0.00 -> 2.23 mm, vias 0 -> 1
- net GND: track 3.26 -> 4.52 mm, vias 14 -> 18
- net +3V3: track 44.3 -> 45.3 mm, vias 5 -> 3
- net Net-(T3-E): track 8.07 -> 8.73 mm, vias 1 -> 0
- net Net-(D5-K): track 5.09 -> 5.71 mm
- net /BUS_V: track 13.2 -> 13.7 mm
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
Commit message: finally standardize selected parts on all boards
Parts:
- D6, D7: footprint Diode_SMD:D_SOD-123 -> Diode_SMD:D_MiniMELF
- R13: value 6,2k -> 6k2
- R25: value 24R 1W -> 24R 1W
- moved R4 1.30 mm to (143.8, 101.9)
- moved D7 0.26 mm to (137.4, 110.0)
- moved C3 0.25 mm to (146.6, 101.9)
- moved R1 0.25 mm to (146.6, 103.9)
Routing:
- net Net-(D5-K): track 5.71 -> 4.51 mm
- net Net-(T3-C): track 4.55 -> 5.50 mm

Commit message: final for manufacturing
Parts:
- C1: value 100µ/35V -> 100u/35V
- C13, C14: value 47µ/10V -> 47u/10V
- C7: value 4.7µ/35V -> 4.7u/35V
- R16: value 88k7 -> 51k
- R25: footprint Resistor_SMD:R_1206_3216Metric -> Resistor_SMD:R_2512_6332Metric
- moved R25 0.89 mm to (136.7, 108.7)
Changed lines of the file:
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@@
 			)
 		)
-		(property "Value" "47µ/10V"
+		(property "Value" "47u/10V"
 			(at 0 1.85 0)
 			(layer "F.Fab")
@@
 			)
 		)
-		(property "Value" "88k7"
+		(property "Value" "51k"
 			(at 0 1.65 180)
 			(layer "F.Fab")
@@
 			)
 		)
-		(property "Value" "4.7µ/35V"
+		(property "Value" "4.7u/35V"
 			(at 0 1.68 90)
 			(layer "F.Fab")
@@
 			)
 		)
-		(property "Value" "100µ/35V"
+		(property "Value" "100u/35V"
 			(at 0 4.35 90)
 			(layer "F.Fab")
@@
 			)
 		)
-		(property "Value" "47µ/10V"
+		(property "Value" "47u/10V"
 			(at 0 1.85 0)
 			(layer "F.Fab")
@@
 		(tags "resistor")
 		(property "Reference" "R5"
-			(at -2.6751 0.7904 0)
+			(at 0.1189 -8.3536 0)
 			(layer "B.SilkS")
 			(effects
@@
 		(tags "capacitor")
 		(property "Reference" "C4"
-			(at 2.6751 1.5346 180)
+			(at -0.1189 9.9166 180)
 			(layer "B.SilkS")
 			(effects
@@
 		)
 	)
-	(footprint "Resistor_SMD:R_1206_3216Metric"
+	(footprint "Resistor_SMD:R_2512_6332Metric"
 		(layer "B.Cu")
-		(at 136.652 107.823 90)
-		(descr "Resistor SMD 1206 (3216 Metric), square (rectangular) end terminal, IPC_7351 nominal, (Body size source: IPC-SM-782 page 72, https://www.pcb-3d.com/wordpress/wp-content/uploads/ipc-sm-782a_amendment_1_and_2.pdf), generated with kicad-footprint-generator")
+		(at 136.652 108.712 90)
+		(descr "Resistor SMD 2512 (6332 Metric), square (rectangular) end terminal, IPC_7351 nominal, (Body size source: IPC-SM-782 page 72, https://www.pcb-3d.com/wordpress/wp-content/uploads/ipc-sm-782a_amendment_1_and_2.pdf), generated with kicad-footprint-generator")
 		(tags "resistor")
 		(property "Reference" "R25"
-			(at 2.921 0 0)
+			(at 5.588 1.524 -90)
 			(layer "B.SilkS")
 			(effects
@@
 		)
 		(property "Value" "24R 1W"
-			(at 0 -1.82 90)
+			(at 0 -2.62 -90)
 			(layer "B.Fab")
 			(effects
@@
 			)
 		)
-		(property "Footprint" "Resistor_SMD:R_1206_3216Metric"
+		(property "Footprint" "Resistor_SMD:R_2512_6332Metric"
 			(at 0 0 -90)
 			(unlocked yes)
@@
 		(attr smd)
 		(fp_line
-			(start 0.727064 -0.91)
-			(end -0.727064 -0.91)
+			(start 2.177064 -1.71)
+			(end -2.177064 -1.71)
 			(stroke
 				(width 0.12)
@@
 		)
 		(fp_line
-			(start 0.727064 0.91)
-			(end -0.727064 0.91)
+			(start 2.177064 1.71)
+			(end -2.177064 1.71)
 			(stroke
 				(width 0.12)
@@
 		)
 		(fp_line
-			(start 2.28 -1.12)
-			(end 2.28 1.12)
+			(start 3.82 -1.92)
+			(end 3.82 1.92)
 			(stroke
 				(width 0.05)
@@
 		)
 		(fp_line
-			(start -2.28 -1.12)
-			(end 2.28 -1.12)
+			(start -3.82 -1.92)
+			(end 3.82 -1.92)
 			(stroke
 				(width 0.05)
@@
 		)
 		(fp_line
-			(start 2.28 1.12)
-			(end -2.28 1.12)
+			(start 3.82 1.92)
+			(end -3.82 1.92)
 			(stroke
 				(width 0.05)
@@
 		)
 		(fp_line
-			(start -2.28 1.12)
-			(end -2.28 -1.12)
+			(start -3.82 1.92)
+			(end -3.82 -1.92)
 			(stroke
 				(width 0.05)
@@
 		)
 		(fp_line
-			(start 1.6 -0.8)
-			(end 1.6 0.8)
+			(start 3.15 -1.6)
+			(end 3.15 1.6)
 			(stroke
 				(width 0.1)
@@
 		)
 		(fp_line
-			(start -1.6 -0.8)
-			(end 1.6 -0.8)
+			(start -3.15 -1.6)
+			(end 3.15 -1.6)
 			(stroke
 				(width 0.1)
@@
 		)
 		(fp_line
-			(start 1.6 0.8)
-			(end -1.6 0.8)
+			(start 3.15 1.6)
+			(end -3.15 1.6)
 			(stroke
 				(width 0.1)
@@
 		)
 		(fp_line
-			(start -1.6 0.8)
-			(end -1.6 -0.8)
+			(start -3.15 1.6)
+			(end -3.15 -1.6)
 			(stroke
 				(width 0.1)
@@
 		)
 		(fp_text user "${REFERENCE}"
-			(at 0 0 90)
+			(at 0 0 -90)
 			(layer "B.Fab")
 			(effects
 				(font
-					(size 0.8 0.8)
-					(thickness 0.12)
+					(size 1 1)
+					(thickness 0.15)
 				)
 				(justify mirror)
@@
 		)
 		(pad "1" smd roundrect
-			(at -1.4625 0 90)
-			(size 1.125 1.75)
+			(at -2.9625 0 90)
+			(size 1.225 3.35)
 			(layers "B.Cu" "B.Paste" "B.Mask")
-			(roundrect_rratio 0.222222)
+			(roundrect_rratio 0.204082)
 			(net 17 "Net-(T3-E)")
 			(pintype "passive")
 		)
 		(pad "2" smd roundrect
-			(at 1.4625 0 90)
-			(size 1.125 1.75)
+			(at 2.9625 0 90)
+			(size 1.225 3.35)
 			(layers "B.Cu" "B.Paste" "B.Mask")
-			(roundrect_rratio 0.222222)
+			(roundrect_rratio 0.204082)
 			(net 20 "/HEAT")
 			(pintype "passive")
 		)
-		(model "${KICAD8_3DMODEL_DIR}/Resistor_SMD.3dshapes/R_1206_3216Metric.wrl"
+		(model "${KICAD8_3DMODEL_DIR}/Resistor_SMD.3dshapes/R_2512_6332Metric.wrl"
 			(offset
 				(xyz 0 0 0)
@@
 		(tags "resistor")
 		(property "Reference" "R6"
-			(at -4.3261 -0.2436 0)
+			(at 0.1189 -9.1336 0)
 			(layer "B.SilkS")
 			(effects
@@
 		(tags "SOD-123")
 		(property "Reference" "D4"
-			(at 0 2 0)
+			(at 3.429 0 0)
 			(layer "B.SilkS")
 			(effects
@@
 		(tags "SOT TO_SOT_SMD")
 		(property "Reference" "T3"
-			(at 2.5736 0.1119 180)
+			(at 6.3836 0.6199 180)
 			(layer "B.SilkS")
 			(effects
@@
 	)
 	(via
-		(at 137.795 110.363)
+		(at 137.922 110.236)
 		(size 0.6)
 		(drill 0.3)
@@
 	)
 	(segment
-		(start 136.652 111.125)
-		(end 137.6911 112.1641)
+		(start 137.6911 113.5611)
+		(end 137.6911 114.1566)
 		(width 0.6096)
 		(layer "B.Cu")
@@
 	)
 	(segment
-		(start 138.2864 107.6511)
-		(end 136.652 109.2855)
+		(start 136.652 109.22)
+		(end 138.2209 107.6511)
 		(width 0.4064)
 		(layer "B.Cu")
@@
 	)
 	(segment
-		(start 139.4001 107.6511)
-		(end 138.2864 107.6511)
+		(start 138.2209 107.6511)
+		(end 139.4001 107.6511)
 		(width 0.4064)
 		(layer "B.Cu")
@@
 	)
 	(segment
-		(start 136.652 109.2855)
-		(end 136.652 111.125)
+		(start 136.652 111.6745)
+		(end 136.652 112.522)
 		(width 0.6096)
 		(layer "B.Cu")
@@
 	)
 	(segment
-		(start 137.6911 112.1641)
-		(end 137.6911 114.1566)
+		(start 136.652 112.522)
+		(end 137.6911 113.5611)
 		(width 0.6096)
 		(layer "B.Cu")
 		(net 17)
+	)
+	(segment
+		(start 136.652 111.6745)
+		(end 136.652 109.22)
+		(width 0.4064)
+		(layer "B.Cu")
+		(net 17)

Commit message: update bb_pwr_knx_v-measure
Parts:
- C9: value 15n -> 100n
Changed lines of the file:
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@@
 			)
 		)
-		(property "Value" "15n"
+		(property "Value" "100n"
 			(at 0 1.68 0)
 			(layer "F.Fab")
